File: hardware/lobby/lobby.kicad_pcb (KiCad board)
At the start: 0 parts

Commit message: start routing mezzanine
making a progress capture before trying to cram a lot of signals onto just one hirose connector...
Parts:
- added C1: 10u, Capacitor_SMD:C_0805_2012Metric, F.Cu at (139.7, 63.5)
- added C2: 47 uF / 6.3V, Capacitor_SMD:C_0805_2012Metric, F.Cu at (174.2, 131.1)
- added C3: 10 uF / 25V, Capacitor_SMD:C_0805_2012Metric, F.Cu at (183.4, 121.9)
- added J1: Micro_SD_Card_Det, cm4crypto:SDCARD_MOLEX_503398-1892, F.Cu at (129.9, 71.9)
- added J2: Conn_01x22_Female, Connector_FFC-FPC:Hirose_FH12-22S-0.5SH_1x22-1MP_P0.50mm_Horizontal, F.Cu at (137.6, 123.9)
- added JP1: SolderJumper_2_Open, Jumper:SolderJumper-2_P1.3mm_Open_TrianglePad1.0x1.5mm, F.Cu at (181.6, 63.8)
- added JP2: SolderJumper_2_Open, Jumper:SolderJumper-2_P1.3mm_Open_TrianglePad1.0x1.5mm, F.Cu at (168.0, 73.0)
- added JP3: SolderJumper_2_Open, Jumper:SolderJumper-2_P1.3mm_Open_TrianglePad1.0x1.5mm, F.Cu at (168.0, 76.5)
- added JP4: SolderJumper_2_Open, Jumper:SolderJumper-2_P1.3mm_Open_TrianglePad1.0x1.5mm, F.Cu at (172.3, 73.0)
- added JP5: Jumper_2_Bridged, Jumper:SolderJumper-2_P1.3mm_Bridged_Pad1.0x1.5mm, F.Cu at (177.3, 63.8)
- added JP6: SolderJumper_2_Open, Jumper:SolderJumper-2_P1.3mm_Open_TrianglePad1.0x1.5mm, F.Cu at (174.0, 68.8)
- added Module1: ComputeModule4-CM4, cm4crypto:Raspberry-Pi-4-Compute-Module, F.Cu at (46.0, 114.2)
- added Module2: cm4-module-A, cm4crypto:DF40C-100DS-0.4V(51), F.Cu at (88.1, 142.2)
- added Module3: cm4-module-B, cm4crypto:DF40C-100DS-0.4V(51), F.Cu at (88.1, 163.7)
- added R1: 2.2K, Resistor_SMD:R_0603_1608Metric, F.Cu at (85.2, 63.2)
- added R2: 2.2K, Resistor_SMD:R_0603_1608Metric, F.Cu at (43.9, 119.6)
- added R3: nf, Resistor_SMD:R_0402_1005Metric, F.Cu at (123.9, 85.3)
- added R4: nf, Resistor_SMD:R_0402_1005Metric, F.Cu at (138.9, 66.0)
- added R5: 12K 1%, Resistor_SMD:R_0402_1005Metric, F.Cu at (143.4, 63.0)
- added R6: 2.2k, Resistor_SMD:R_0603_1608Metric, F.Cu at (178.1, 66.8)
- added R7: R, Resistor_SMD:R_0603_1608Metric, F.Cu at (173.9, 133.8)
- added SW1: SW_Push, cm4crypto:EVQ-P7C01P, F.Cu at (168.8, 69.1)
- added SW2: SW_SPST, cm4crypto:cus-12b, F.Cu at (170.4, 65.0)
- added U1: RT9742GGJ5, Package_TO_SOT_SMD:SOT-23-5, F.Cu at (125.0, 82.1)
- added U2: M.2-keyM, cm4crypto:M.2 - M - MDT420M01002, F.Cu at (221.2, 69.1)
- added U3: MYLSM00502ERPL, cm4crypto:MYLSM00502ERPL, F.Cu at (172.7, 128.8)
- added U4: FSUSB42MX, Package_SO:MSOP-10_3x3mm_P0.5mm, F.Cu at (45.5, 133.8)
Other:
- copper layers 0 -> 2
