File: hardware/lobby/lobby.kicad_pcb (KiCad board)
At the start: 4 copper layers, 85 x 56 mm, 40 parts, among them J1 THD-02-R, J2 THD-20-R, J3 Micro_SD_Card_Det, J4 Conn_01x22_Female, SW1 SW_Push, SW2 SW_SPST, U1 RT9742GGJ5, U2 M.2-keyM, U3 MYLSM00502ERPL, U4 FSUSB42MX

Commit message: update silkscreen
Parts:
- added REF**: subluminal-logo, cm4crypto:subluminal-logo, B.Cu at (98.0, 42.0)
- SW1: value SW_Push -> SW_SPST; footprint cm4crypto:EVQ-P7C01P -> cm4crypto:cus-12b
- moved SW1 39.1 mm to (34.5, 21.7)
Routing:
- net /nRPIBOOT: track 39.8 -> 76.9 mm, vias 1 -> 3
- net GND: vias 162 -> 160
Other:
- board text added: "1.8V"
- board text added: "3.3V"
- board text added: "BOOT"
- board text added: "DEV"
- board text added: "DISABLE Bluetooth"
- board text added: "DISABLE WiFi"
- board text added: "EEPROM Write Protect"
- board text added: "Force BOOT"
- board text added: "GPIO VREF"
- board text added: "GPIO14 (FAN)"
- board text added: "INTERNAL"
- board text added: "OTG"
- board text added: "RPIBOOT"
- board text added: "USB-C"
- board text added: "subluminal.li"
