File: hardware/lobby/lobby.kicad_sch (KiCad schematic)
At the start: 7 parts, among them J1 THD-02-R, J2 THD-20-R

Commit message: update lobby
Parts:
- added H?: MountingHole, MountingHole:MountingHole_2.7mm_M2.5, symbol Mechanical:MountingHole
- renumbered R8 to R3, R9 to R4

Commit message: Update lobby.kicad_sch
Parts:
- added H2: MountingHole, MountingHole:MountingHole_2.7mm_M2.5, symbol Mechanical:MountingHole
- gave numbers to parts that had none: 1
Changed lines of the file:
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@@
   (symbol (lib_id "Mechanical:MountingHole") (at 179.07 168.91 0) (unit 1)
     (in_bom yes) (on_board yes)
-    (property "Reference" "H?" (id 0) (at 181.61 167.767 0)
+    (property "Reference" "H1" (id 0) (at 181.61 167.767 0)
       (effects (font (size 1.27 1.27)) (justify left))
     )
@@
     )
     (property "Datasheet" "~" (id 3) (at 179.07 168.91 0)
+      (effects (font (size 1.27 1.27)) hide)
+    )
+  )
+  (symbol (lib_id "Mechanical:MountingHole") (at 179.07 173.99 0) (unit 1)
+    (in_bom yes) (on_board yes)
+    (property "Reference" "H2" (id 0) (at 181.61 172.847 0)
+      (effects (font (size 1.27 1.27)) (justify left))
+    )
+    (property "Value" "MountingHole" (id 1) (at 181.61 175.133 0)
+      (effects (font (size 1.27 1.27)) (justify left))
+    )
+    (property "Footprint" "MountingHole:MountingHole_2.7mm_M2.5" (id 2) (at 179.07 173.99 0)
+      (effects (font (size 1.27 1.27)) hide)
+    )
+    (property "Datasheet" "~" (id 3) (at 179.07 173.99 0)
       (effects (font (size 1.27 1.27)) hide)
     )
@@
     )
     (path "/7a70a0f1-e28b-45e1-81d6-e8a736d785e2"
-      (reference "H?") (unit 1) (value "MountingHole") (footprint "MountingHole:MountingHole_2.7mm_M2.5")
+      (reference "H1") (unit 1) (value "MountingHole") (footprint "MountingHole:MountingHole_2.7mm_M2.5")
+    )
+    (path "/5c613380-e300-4605-8332-4dd58f76d9ad"
+      (reference "H2") (unit 1) (value "MountingHole") (footprint "MountingHole:MountingHole_2.7mm_M2.5")
     )
     (path "/335cd064-cc6e-45d8-b956-940048207657"
