File: hardware/mezzanine/mezzanine.kicad_pcb (KiCad board)
At the start: 0 parts

Commit message: start routing mezzanine
making a progress capture before trying to cram a lot of signals onto just one hirose connector...
Parts:
- added C1: 10u, Capacitor_SMD:C_0805_2012Metric, F.Cu at (267.6, 77.6)
- added C10: 100n, Capacitor_SMD:C_0402_1005Metric, F.Cu at (255.7, 90.7)
- added C11: 100n, Capacitor_SMD:C_0402_1005Metric, F.Cu at (241.7, 99.2)
- added C12: 100n, Capacitor_SMD:C_0402_1005Metric, F.Cu at (262.4, 83.1)
- added C13: 100n, Capacitor_SMD:C_0402_1005Metric, F.Cu at (244.6, 99.2)
- added C14: 100n, Capacitor_SMD:C_0402_1005Metric, F.Cu at (260.9, 86.2)
- added C15: 100n, Capacitor_SMD:C_0402_1005Metric, F.Cu at (206.9, 100.1)
- added C16: 100n, Capacitor_SMD:C_0402_1005Metric, F.Cu at (194.1, 133.9)
- added C17: 100n, Capacitor_SMD:C_0402_1005Metric, F.Cu at (194.1, 132.0)
- added C2: 100uF, Capacitor_Tantalum_SMD:CP_EIA-7343-31_Kemet-D, F.Cu at (237.2, 95.1)
- added C3: 10u, Capacitor_SMD:C_0805_2012Metric, F.Cu at (263.2, 77.6)
- added C4: 10u, Capacitor_SMD:C_0805_2012Metric, F.Cu at (244.4, 93.7)
- added C5: 10u, Capacitor_SMD:C_0805_2012Metric, F.Cu at (252.1, 91.2)
- added C6: 10u, Capacitor_SMD:C_0805_2012Metric, F.Cu at (244.4, 96.7)
- added C7: 10u, Capacitor_SMD:C_0805_2012Metric, F.Cu at (263.2, 80.6)
- added C8: 10u, Capacitor_SMD:C_0805_2012Metric, F.Cu at (257.2, 86.8)
- added C9: 100n, Capacitor_SMD:C_0402_1005Metric, F.Cu at (248.0, 97.2)
- added D1: LED Red, LED_SMD:LED_0603_1608Metric, F.Cu at (180.7, 81.2)
- added D2: LED Green, LED_SMD:LED_0603_1608Metric, F.Cu at (184.9, 77.4)
- added H1: MountingHole, MountingHole:MountingHole_2.7mm_M2.5, F.Cu at (23.5, 23.5)
- added H2: MountingHole, MountingHole:MountingHole_2.7mm_M2.5, F.Cu at (23.5, 72.5)
- added H4: MountingHole, MountingHole:MountingHole_2.7mm_M2.5, F.Cu at (81.5, 23.5)
- added J1: USB_A, cm4crypto:OnShore_USB-A1HSB6, F.Cu at (97.7, 67.0)
- added J2: USB_C, cm4crypto:USB4105-GF-A, F.Cu at (31.2, 76.0)
- added J3: HDMI_D, cm4crypto:HD-RA-DSF12-TR, F.Cu at (46.0, 76.0)
- added J4: HDMI_D, cm4crypto:HD-RA-DSF12-TR, F.Cu at (59.5, 76.0)
- added Module1: cm4-module-A, cm4crypto:DF40C-100DP-0.4V(51), B.Cu at (85.0, 50.0)
- added Module2: cm4-module-B, cm4crypto:DF40C-100DP-0.4V(51), B.Cu at (55.0, 60.0)
- added R1: 15K 1%, Resistor_SMD:R_0402_1005Metric, F.Cu at (250.9, 93.7)
- added R2: 5.1k, Resistor_SMD:R_0603_1608Metric, F.Cu at (238.3, 99.4)
- added R3: 5.1k, Resistor_SMD:R_0603_1608Metric, F.Cu at (234.3, 99.3)
- added R4: 470R, Resistor_SMD:R_0402_1005Metric, F.Cu at (219.2, 81.1)
- added R5: 470R, Resistor_SMD:R_0402_1005Metric, F.Cu at (222.1, 77.1)
- added R6: 1k, Resistor_SMD:R_0402_1005Metric, F.Cu at (188.4, 77.1)
- added R7: 1k, Resistor_SMD:R_0603_1608Metric, F.Cu at (184.7, 81.2)
- added TP1: TestPoint, TestPoint:TestPoint_Pad_2.0x2.0mm, F.Cu at (180.7, 84.5)
- added U1: AP22653W6, Package_TO_SOT_SMD:SOT-23-6, F.Cu at (252.4, 87.5)
- added U2: TPD4EUSB30, Package_SON:USON-10_2.5x1.0mm_P0.5mm, F.Cu at (248.0, 94.2)
- added U3: TPD4EUSB30, Package_SON:USON-10_2.5x1.0mm_P0.5mm, F.Cu at (199.7, 108.3)
- added U4: TPD4EUSB30, Package_SON:USON-10_2.5x1.0mm_P0.5mm, F.Cu at (219.2, 78.1)
- added U5: MagJack-A70-112-331N126, cm4crypto:TRJG0926HENL, F.Cu at (97.0, 30.2)
- added U6: RT9742SNGV, Package_TO_SOT_SMD:SOT-23, F.Cu at (190.2, 133.2)
- added U7: 74LVC1G07SE-7, Package_TO_SOT_SMD:SOT-353_SC-70-5, F.Cu at (180.8, 78.0)
Other:
- board outline added: 85 x 56 mm
- copper layers 0 -> 2
