File: hardware/mezzanine/mezzanine.kicad_pcb (KiCad board)
At the start: 4 copper layers, 85 x 56 mm, 34 parts, among them J1 USB_A, J2 USB_C, J3 HDMI_D, J4 HDMI_D, U1 AP22653W6, U2 TPD4EUSB30, U3 TPD4EUSB30, U4 TPD4EUSB30, U5 MagJack-A70-112-331N126, U6 RT9742SNGV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

Commit message: pushing local changes
including prelim docs
Parts:
- U1: value AP22653W6 -> AP22652AW6-7
Changed lines of the file:
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@@
       (effects (font (size 1 1) (thickness 0.15)))
     )
-    (fp_text value "AP22653W6" (at 0 4.5 90) (layer "F.Fab")
+    (fp_text value "AP22652AW6-7" (at 0 4.5 90) (layer "F.Fab")
       (effects (font (size 1 1) (thickness 0.15)))
     )
