File: hardware/mezzanine/sheets/gpio.kicad_sch (KiCad schematic)
At the start: 1 part

Commit message: start routing mezzanine
making a progress capture before trying to cram a lot of signals onto just one hirose connector...
Parts:
- removed J?: THD-20-R, CM4IO:rpi-40-just-power, symbol Connector_Generic:Conn_02x20_Odd_Even
Other:
- note removed: "40Way GPIO Header"
- note removed: "gpio header is only supplying compatibility with POE hats..."
- note removed: "providing gpio4 for fan control"
Changed lines of the file:
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@@
 (kicad_sch (version 20210406) (generator eeschema)
   (paper "A4")
-  (junction (at 138.43 54.61) (diameter 1.016) (color 0 0 0 0))
-  (junction (at 139.7 85.09) (diameter 1.016) (color 0 0 0 0))
-  (junction (at 139.7 102.87) (diameter 1.016) (color 0 0 0 0))
-  (junction (at 154.94 54.61) (diameter 1.016) (color 0 0 0 0))
-  (junction (at 154.94 69.85) (diameter 1.016) (color 0 0 0 0))
-  (junction (at 154.94 77.47) (diameter 1.016) (color 0 0 0 0))
-  (junction (at 154.94 90.17) (diameter 1.016) (color 0 0 0 0))
-  (junction (at 154.94 95.25) (diameter 1.016) (color 0 0 0 0))
-  (wire (pts (xy 129.54 57.15) (xy 140.97 57.15))
-    (stroke (width 0) (type solid) (color 0 0 0 0))
-  )
-  (wire (pts (xy 129.54 59.69) (xy 140.97 59.69))
-    (stroke (width 0) (type solid) (color 0 0 0 0))
-  )
-  (wire (pts (xy 129.54 62.23) (xy 140.97 62.23))
-    (stroke (width 0) (type solid) (color 0 0 0 0))
-  )
-  (wire (pts (xy 132.08 54.61) (xy 138.43 54.61))
-    (stroke (width 0) (type solid) (color 0 0 0 0))
-  )
-  (wire (pts (xy 138.43 54.61) (xy 138.43 74.93))
-    (stroke (width 0) (type solid) (color 0 0 0 0))
-  )
-  (wire (pts (xy 138.43 74.93) (xy 140.97 74.93))
-    (stroke (width 0) (type solid) (color 0 0 0 0))
-  )
-  (wire (pts (xy 139.7 64.77) (xy 139.7 85.09))
-    (stroke (width 0) (type solid) (color 0 0 0 0))
-  )
-  (wire (pts (xy 139.7 85.09) (xy 139.7 102.87))
-    (stroke (width 0) (type solid) (color 0 0 0 0))
-  )
-  (wire (pts (xy 139.7 85.09) (xy 140.97 85.09))
-    (stroke (width 0) (type solid) (color 0 0 0 0))
-  )
-  (wire (pts (xy 139.7 102.87) (xy 139.7 104.14))
-    (stroke (width 0) (type solid) (color 0 0 0 0))
-  )
-  (wire (pts (xy 139.7 102.87) (xy 140.97 102.87))
-    (stroke (width 0) (type solid) (color 0 0 0 0))
-  )
-  (wire (pts (xy 140.97 54.61) (xy 138.43 54.61))
-    (stroke (width 0) (type solid) (color 0 0 0 0))
-  )
-  (wire (pts (xy 140.97 64.77) (xy 139.7 64.77))
-    (stroke (width 0) (type solid) (color 0 0 0 0))
-  )
-  (wire (pts (xy 153.67 54.61) (xy 154.94 54.61))
-    (stroke (width 0) (type solid) (color 0 0 0 0))
-  )
-  (wire (pts (xy 153.67 57.15) (xy 154.94 57.15))
-    (stroke (width 0) (type solid) (color 0 0 0 0))
-  )
-  (wire (pts (xy 153.67 59.69) (xy 154.94 59.69))
-    (stroke (width 0) (type solid) (color 0 0 0 0))
-  )
-  (wire (pts (xy 153.67 90.17) (xy 154.94 90.17))
-    (stroke (width 0) (type solid) (color 0 0 0 0))
-  )
-  (wire (pts (xy 153.67 95.25) (xy 154.94 95.25))
-    (stroke (width 0) (type solid) (color 0 0 0 0))
-  )
-  (wire (pts (xy 154.94 54.61) (xy 160.02 54.61))
-    (stroke (width 0) (type solid) (color 0 0 0 0))
-  )
-  (wire (pts (xy 154.94 57.15) (xy 154.94 54.61))
-    (stroke (width 0) (type solid) (color 0 0 0 0))
-  )
-  (wire (pts (xy 154.94 59.69) (xy 154.94 69.85))
-    (stroke (width 0) (type solid) (color 0 0 0 0))
-  )
-  (wire (pts (xy 154.94 69.85) (xy 153.67 69.85))
-    (stroke (width 0) (type solid) (color 0 0 0 0))
-  )
-  (wire (pts (xy 154.94 69.85) (xy 154.94 77.47))
-    (stroke (width 0) (type solid) (color 0 0 0 0))
-  )
-  (wire (pts (xy 154.94 77.47) (xy 153.67 77.47))
-    (stroke (width 0) (type solid) (color 0 0 0 0))
-  )
-  (wire (pts (xy 154.94 90.17) (xy 154.94 77.47))
-    (stroke (width 0) (type solid) (color 0 0 0 0))
-  )
-  (wire (pts (xy 154.94 95.25) (xy 154.94 90.17))
-    (stroke (width 0) (type solid) (color 0 0 0 0))
-  )
-  (wire (pts (xy 154.94 95.25) (xy 154.94 104.14))
-    (stroke (width 0) (type solid) (color 0 0 0 0))
-  )
-  (polyline (pts (xy 127 44.45) (xy 127 110.49))
-    (stroke (width 0) (type solid) (color 0 0 0 0))
-  )
-  (polyline (pts (xy 127 110.49) (xy 167.64 110.49))
-    (stroke (width 0) (type solid) (color 0 0 0 0))
-  )
-  (polyline (pts (xy 167.64 44.45) (xy 127 44.45))
-    (stroke (width 0) (type solid) (color 0 0 0 0))
-  )
-  (polyline (pts (xy 167.64 44.45) (xy 167.64 110.49))
-    (stroke (width 0) (type solid) (color 0 0 0 0))
-  )
-  (text "40Way GPIO Header" (at 132.08 49.53 0)
-    (effects (font (size 2.007 2.007)) (justify left bottom))
-  )
-  (text "providing gpio4 for fan control" (at 135.89 66.04 270)
-    (effects (font (size 1.27 1.27)) (justify right bottom))
-  )
-  (text "gpio header is only supplying compatibility with POE hats..."
-    (at 173.99 139.7 0)
-    (effects (font (size 1.27 1.27)) (justify right bottom))
-  )
-  (label "GPIO2" (at 135.89 57.15 180)
-    (effects (font (size 1.27 1.27)) (justify right bottom))
-  )
-  (label "GPIO3" (at 135.89 59.69 180)
-    (effects (font (size 1.27 1.27)) (justify right bottom))
-  )
-  (label "GPIO4" (at 135.89 62.23 180)
-    (effects (font (size 1.27 1.27)) (justify right bottom))
-  )
-  (label "+3.3v" (at 137.16 54.61 180)
-    (effects (font (size 1.27 1.27)) (justify right bottom))
-  )
-  (label "+5v" (at 158.75 54.61 180)
-    (effects (font (size 1.27 1.27)) (justify right bottom))
-  )
-  (symbol (lib_id "power:GND") (at 139.7 104.14 0) (unit 1)
-    (in_bom yes) (on_board yes)
-    (property "Reference" "#PWR?" (id 0) (at 139.7 110.49 0)
-      (effects (font (size 1.27 1.27)) hide)
-    )
-    (property "Value" "GND" (id 1) (at 139.827 108.5342 0))
-    (property "Footprint" "" (id 2) (at 139.7 104.14 0)
-      (effects (font (size 1.27 1.27)) hide)
-    )
-    (property "Datasheet" "" (id 3) (at 139.7 104.14 0)
-      (effects (font (size 1.27 1.27)) hide)
-    )
-    (pin "1")
-  )
-  (symbol (lib_id "power:GND") (at 154.94 104.14 0) (unit 1)
-    (in_bom yes) (on_board yes)
-    (property "Reference" "#PWR?" (id 0) (at 154.94 110.49 0)
-      (effects (font (size 1.27 1.27)) hide)
-    )
-    (property "Value" "GND" (id 1) (at 155.067 108.5342 0))
-    (property "Footprint" "" (id 2) (at 154.94 104.14 0)
-      (effects (font (size 1.27 1.27)) hide)
-    )
-    (property "Datasheet" "" (id 3) (at 154.94 104.14 0)
-      (effects (font (size 1.27 1.27)) hide)
-    )
-    (pin "1")
-  )
-  (symbol (lib_id "Connector_Generic:Conn_02x20_Odd_Even") (at 146.05 77.47 0) (unit 1)
-    (in_bom yes) (on_board yes)
-    (property "Reference" "J?" (id 0) (at 154.94 52.07 0))
-    (property "Value" "THD-20-R" (id 1) (at 147.32 51.4096 0))
-    (property "Footprint" "CM4IO:rpi-40-just-power" (id 2) (at 146.05 77.47 0)
-      (effects (font (size 1.27 1.27)) hide)
-    )
-    (property "Datasheet" "https://www.toby.co.uk/uploads/publications/1673.pdf" (id 3) (at 146.05 77.47 0)
-      (effects (font (size 1.27 1.27)) hide)
-    )
-    (property "Field4" "Toby" (id 4) (at 146.05 77.47 0)
-      (effects (font (size 1.27 1.27)) hide)
-    )
-    (property "Field5" "THD-20-R" (id 5) (at 146.05 77.47 0)
-      (effects (font (size 1.27 1.27)) hide)
-    )
-    (property "Field6" "THD-20-R" (id 6) (at 146.05 77.47 0)
-      (effects (font (size 1.27 1.27)) hide)
-    )
-    (property "Field7" "Toby" (id 7) (at 146.05 77.47 0)
-      (effects (font (size 1.27 1.27)) hide)
-    )
-    (property "Field8" "UCON00511" (id 8) (at 146.05 77.47 0)
-      (effects (font (size 1.27 1.27)) hide)
-    )
-    (property "Part Description" "PinHeader_2x20_P2.54mm_Vertical" (id 9) (at 146.05 77.47 0)
-      (effects (font (size 1.27 1.27)) hide)
-    )
-    (pin "1")
-    (pin "10")
-    (pin "11")
-    (pin "12")
-    (pin "13")
-    (pin "14")
-    (pin "15")
-    (pin "16")
-    (pin "17")
-    (pin "18")
-    (pin "19")
-    (pin "2")
-    (pin "20")
-    (pin "21")
-    (pin "22")
-    (pin "23")
-    (pin "24")
-    (pin "25")
-    (pin "26")
-    (pin "27")
-    (pin "28")
-    (pin "29")
-    (pin "3")
-    (pin "30")
-    (pin "31")
-    (pin "32")
-    (pin "33")
-    (pin "34")
-    (pin "35")
-    (pin "36")
-    (pin "37")
-    (pin "38")
-    (pin "39")
-    (pin "4")
-    (pin "40")
-    (pin "5")
-    (pin "6")
-    (pin "7")
-    (pin "8")
-    (pin "9")
-  )
 )
