File: hardware/mezzanine/sheets/hdmi.kicad_sch (KiCad schematic)
At the start: 5 parts

Commit message: start routing mezzanine
making a progress capture before trying to cram a lot of signals onto just one hirose connector...
Parts:
- J4, J5: renamed from J?; footprint CM4IO:HD-RA-DSF12-TR -> cm4crypto:HD-RA-DSF12-TR
- gave numbers to parts that had none: 3
Connections:
- net HDMI0_CK_N renamed HDMI0_CLK_N
- net HDMI0_CK_P renamed HDMI0_CLK_P
- net HDMI0_D0_N renamed HDMI0_TX0_N
- net HDMI0_D0_P renamed HDMI0_TX0_P
- net HDMI0_D1_N renamed HDMI0_TX1_N
- net HDMI0_D1_P renamed HDMI0_TX1_P
- net HDMI0_D2_N renamed HDMI0_TX2_N
- net HDMI0_D2_P renamed HDMI0_TX2_P
- net HDMI1_CK_N renamed HDMI1_CLK_N
- net HDMI1_CK_P renamed HDMI1_CLK_P
- net HDMI1_D0_N renamed HDMI1_TX0_N
- net HDMI1_D0_P renamed HDMI1_TX0_P
- net HDMI1_D1_N renamed HDMI1_TX1_N
- net HDMI1_D1_P renamed HDMI1_TX1_P
- net HDMI1_D2_N renamed HDMI1_TX2_N
- net HDMI1_D2_P renamed HDMI1_TX2_P

Commit message: finished mezzanine signal routing
Parts:
- C8: renamed from C16; footprint Capacitor_SMD:C_0402_1005Metric -> Capacitor_SMD:C_0603_1608Metric; Field4 Farnell -> (none); Field5 2611911 -> (none); Field6 RM EMK105 B7104KV-F -> (none); Field7 TAIYO YUDEN EUROPE GMBH -> (none); Field8 110091611 -> (none); Part Description 0.1uF 10% 16V Ceramic Capacitor X7R 0402 (1005 Metric) -> (none)
- C9: renamed from C17; footprint Capacitor_SMD:C_0402_1005Metric -> Capacitor_SMD:C_0603_1608Metric; Field4 Farnell -> (none); Field5 2611911 -> (none); Field6 RM EMK105 B7104KV-F -> (none); Field7 TAIYO YUDEN EUROPE GMBH -> (none); Field8 110091611 -> (none); Part Description 0.1uF 10% 16V Ceramic Capacitor X7R 0402 (1005 Metric) -> (none)
- renumbered J4 to J3, J5 to J4
Connections:
- net HDMI0_CEC: now also J3.15 (CEC); no longer J4.15 (CEC)
- net HDMI0_CLK_N: now also J3.14 (CK-); no longer J4.14 (CK-)
- net HDMI0_CLK_P: now also J3.12 (CK+); no longer J4.12 (CK+)
- net HDMI0_HOTPLUG: now also J3.1 (HPD/HEAC-); no longer J4.1 (HPD/HEAC-)
- net HDMI0_SCL: now also J3.17 (SCL); no longer J4.17 (SCL)
- net HDMI0_SDA: now also J3.18 (SDA); no longer J4.18 (SDA)
- net HDMI0_TX0_N: now also J3.11 (D0-); no longer J4.11 (D0-)
- net HDMI0_TX0_P: now also J3.9 (D0+); no longer J4.9 (D0+)
- net HDMI0_TX1_N: now also J3.8 (D1-); no longer J4.8 (D1-)
- net HDMI0_TX1_P: now also J3.6 (D1+); no longer J4.6 (D1+)
- net HDMI0_TX2_N: now also J3.5 (D2-); no longer J4.5 (D2-)
- net HDMI0_TX2_P: now also J3.3 (D2+); no longer J4.3 (D2+)
- net HDMI1_CEC: now also J4.15 (CEC); no longer J3.15 (CEC)
- net HDMI1_CLK_N: now also J4.14 (CK-); no longer J3.14 (CK-)
- net HDMI1_CLK_P: now also J4.12 (CK+); no longer J3.12 (CK+)
- net HDMI1_HOTPLUG: now also J4.1 (HPD/HEAC-); no longer J3.1 (HPD/HEAC-)
- net HDMI1_SCL: now also J4.17 (SCL); no longer J3.17 (SCL)
- net HDMI1_SDA: now also J4.18 (SDA); no longer J3.18 (SDA)
- net HDMI1_TX0_N: now also J4.11 (D0-); no longer J3.11 (D0-)
- net HDMI1_TX0_P: now also J4.9 (D0+); no longer J3.9 (D0+)
- net HDMI1_TX1_N: now also J4.8 (D1-); no longer J3.8 (D1-)
- net HDMI1_TX1_P: now also J4.6 (D1+); no longer J3.6 (D1+)
- net HDMI1_TX2_N: now also J4.5 (D2-); no longer J3.5 (D2-)
- net HDMI1_TX2_P: now also J4.3 (D2+); no longer J3.3 (D2+)

Commit message: sheet refs relative, copied escalator pinout to lobby
Parts:
- renumbered C9 to C?, C8 to C?, J4 to J?, J3 to J?, U6 to U?
Changed lines of the file:
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@@
   (symbol (lib_id "power:GND") (at 91.44 116.84 0) (unit 1)
     (in_bom yes) (on_board yes)
-    (property "Reference" "#PWR051" (id 0) (at 91.44 123.19 0)
+    (property "Reference" "#PWR?" (id 0) (at 91.44 123.19 0)
       (effects (font (size 1.27 1.27)) hide)
     )
@@
   (symbol (lib_id "power:GND") (at 92.71 161.29 0) (unit 1)
     (in_bom yes) (on_board yes)
-    (property "Reference" "#PWR052" (id 0) (at 92.71 167.64 0)
+    (property "Reference" "#PWR?" (id 0) (at 92.71 167.64 0)
       (effects (font (size 1.27 1.27)) hide)
     )
@@
   (symbol (lib_id "power:GND") (at 104.14 161.29 0) (unit 1)
     (in_bom yes) (on_board yes)
-    (property "Reference" "#PWR053" (id 0) (at 104.14 167.64 0)
+    (property "Reference" "#PWR?" (id 0) (at 104.14 167.64 0)
       (effects (font (size 1.27 1.27)) hide)
     )
@@
   (symbol (lib_id "power:GND") (at 125.73 161.29 0) (unit 1)
     (in_bom yes) (on_board yes)
-    (property "Reference" "#PWR054" (id 0) (at 125.73 167.64 0)
+    (property "Reference" "#PWR?" (id 0) (at 125.73 167.64 0)
       (effects (font (size 1.27 1.27)) hide)
     )
@@
   (symbol (lib_id "power:GND") (at 189.23 115.57 0) (unit 1)
     (in_bom yes) (on_board yes)
-    (property "Reference" "#PWR050" (id 0) (at 189.23 121.92 0)
+    (property "Reference" "#PWR?" (id 0) (at 189.23 121.92 0)
       (effects (font (size 1.27 1.27)) hide)
     )
@@
   (symbol (lib_id "Device:C") (at 92.71 157.48 0) (unit 1)
     (in_bom yes) (on_board yes)
-    (property "Reference" "C8" (id 0) (at 95.631 156.3116 0)
+    (property "Reference" "C?" (id 0) (at 95.631 156.3116 0)
       (effects (font (size 1.27 1.27)) (justify left))
     )
@@
   (symbol (lib_id "Device:C") (at 125.73 157.48 0) (unit 1)
     (in_bom yes) (on_board yes)
-    (property "Reference" "C9" (id 0) (at 128.651 156.3116 0)
+    (property "Reference" "C?" (id 0) (at 128.651 156.3116 0)
       (effects (font (size 1.27 1.27)) (justify left))
     )
@@
   (symbol (lib_id "CM4IO:RT9742SNGV") (at 109.22 157.48 0) (unit 1)
     (in_bom yes) (on_board yes)
-    (property "Reference" "U6" (id 0) (at 111.76 146.939 0))
+    (property "Reference" "U?" (id 0) (at 111.76 146.939 0))
     (property "Value" "RT9742SNGV" (id 1) (at 111.76 149.2504 0))
     (property "Footprint" "Package_TO_SOT_SMD:SOT-23" (id 2) (at 109.22 157.48 0)
@@
   (symbol (lib_id "CM4IO:HDMI_D") (at 96.52 86.36 0) (unit 1)
     (in_bom yes) (on_board yes) (fields_autoplaced)
-    (property "Reference" "J4" (id 0) (at 107.95 85.7249 0)
+    (property "Reference" "J?" (id 0) (at 107.95 85.7249 0)
       (effects (font (size 1.27 1.27)) (justify left))
     )
@@
   (symbol (lib_id "CM4IO:HDMI_D") (at 194.31 85.09 0) (unit 1)
     (in_bom yes) (on_board yes) (fields_autoplaced)
-    (property "Reference" "J3" (id 0) (at 205.74 84.4549 0)
+    (property "Reference" "J?" (id 0) (at 205.74 84.4549 0)
       (effects (font (size 1.27 1.27)) (justify left))
     )

Commit message: addtl hdmi routing
Parts:
- gave numbers to parts that had none: 5
Changed lines of the file:
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@@
+    (stroke (width 0) (type solid) (color 0 0 0 0))
+  )
+  (wire (pts (xy 123.19 35.56) (xy 133.35 35.56))
     (stroke (width 0) (type solid) (color 0 0 0 0))
   )
@@
     (effects (font (size 1.27 1.27)) (justify left bottom))
   )
+  (label "+5v" (at 133.35 35.56 180)
+    (effects (font (size 1.27 1.27)) (justify right bottom))
+  )
   (label "HDMI_5v" (at 134.62 153.67 180)
     (effects (font (size 1.27 1.27)) (justify right bottom))
@@
     (effects (font (size 1.27 1.27)) (justify right))
   )
+  (hierarchical_label "+5v" (shape input) (at 123.19 35.56 180)
+    (effects (font (size 1.27 1.27)) (justify right))
+  )
   (hierarchical_label "HDMI0_TX2_P" (shape input) (at 182.88 64.77 180)
     (effects (font (size 1.27 1.27)) (justify right))
@@
   (symbol (lib_id "power:GND") (at 91.44 116.84 0) (unit 1)
     (in_bom yes) (on_board yes)
-    (property "Reference" "#PWR?" (id 0) (at 91.44 123.19 0)
+    (property "Reference" "#PWR0121" (id 0) (at 91.44 123.19 0)
       (effects (font (size 1.27 1.27)) hide)
     )
@@
   (symbol (lib_id "power:GND") (at 92.71 161.29 0) (unit 1)
     (in_bom yes) (on_board yes)
-    (property "Reference" "#PWR?" (id 0) (at 92.71 167.64 0)
+    (property "Reference" "#PWR0124" (id 0) (at 92.71 167.64 0)
       (effects (font (size 1.27 1.27)) hide)
     )
@@
   (symbol (lib_id "power:GND") (at 104.14 161.29 0) (unit 1)
     (in_bom yes) (on_board yes)
-    (property "Reference" "#PWR?" (id 0) (at 104.14 167.64 0)
+    (property "Reference" "#PWR0123" (id 0) (at 104.14 167.64 0)
       (effects (font (size 1.27 1.27)) hide)
     )
@@
   (symbol (lib_id "power:GND") (at 125.73 161.29 0) (unit 1)
     (in_bom yes) (on_board yes)
-    (property "Reference" "#PWR?" (id 0) (at 125.73 167.64 0)
+    (property "Reference" "#PWR0122" (id 0) (at 125.73 167.64 0)
       (effects (font (size 1.27 1.27)) hide)
     )
@@
   (symbol (lib_id "power:GND") (at 189.23 115.57 0) (unit 1)
     (in_bom yes) (on_board yes)
-    (property "Reference" "#PWR?" (id 0) (at 189.23 121.92 0)
+    (property "Reference" "#PWR0120" (id 0) (at 189.23 121.92 0)
       (effects (font (size 1.27 1.27)) hide)
     )
@@
   (symbol (lib_id "Device:C") (at 92.71 157.48 0) (unit 1)
     (in_bom yes) (on_board yes)
-    (property "Reference" "C?" (id 0) (at 95.631 156.3116 0)
+    (property "Reference" "C8" (id 0) (at 95.631 156.3116 0)
       (effects (font (size 1.27 1.27)) (justify left))
     )
@@
   (symbol (lib_id "Device:C") (at 125.73 157.48 0) (unit 1)
     (in_bom yes) (on_board yes)
-    (property "Reference" "C?" (id 0) (at 128.651 156.3116 0)
+    (property "Reference" "C9" (id 0) (at 128.651 156.3116 0)
       (effects (font (size 1.27 1.27)) (justify left))
     )
@@
   (symbol (lib_id "CM4IO:RT9742SNGV") (at 109.22 157.48 0) (unit 1)
     (in_bom yes) (on_board yes)
-    (property "Reference" "U?" (id 0) (at 111.76 146.939 0))
+    (property "Reference" "U6" (id 0) (at 111.76 146.939 0))
     (property "Value" "RT9742SNGV" (id 1) (at 111.76 149.2504 0))
     (property "Footprint" "Package_TO_SOT_SMD:SOT-23" (id 2) (at 109.22 157.48 0)
@@
   (symbol (lib_id "CM4IO:HDMI_D") (at 96.52 86.36 0) (unit 1)
     (in_bom yes) (on_board yes) (fields_autoplaced)
-    (property "Reference" "J?" (id 0) (at 107.95 85.7249 0)
+    (property "Reference" "J4" (id 0) (at 107.95 85.7249 0)
       (effects (font (size 1.27 1.27)) (justify left))
     )
@@
   (symbol (lib_id "CM4IO:HDMI_D") (at 194.31 85.09 0) (unit 1)
     (in_bom yes) (on_board yes) (fields_autoplaced)
-    (property "Reference" "J?" (id 0) (at 205.74 84.4549 0)
-      (effects (font (size 1.27 1.27)) (justify left))
-    )
+    (property "Reference" "J3" (id 0) (at 205.74 84.4549 0)
+      (effects (font (size 1.27 1.27)) (justify left))
+    )
