File: hardware/mezzanine/sheets/usb.kicad_sch (KiCad schematic)
At the start: 13 parts

Commit message: addtl hdmi routing
Parts:
- R1: renamed from R?; footprint Resistor_SMD:R_0805_2012Metric -> Resistor_SMD:R_0603_1608Metric
- gave numbers to parts that had none: 12
Changed lines of the file:
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@@
   (symbol (lib_id "power:GND") (at 46.99 58.42 0) (unit 1)
     (in_bom yes) (on_board yes)
-    (property "Reference" "#PWR?" (id 0) (at 46.99 64.77 0)
+    (property "Reference" "#PWR0101" (id 0) (at 46.99 64.77 0)
       (effects (font (size 1.27 1.27)) hide)
     )
@@
   (symbol (lib_id "power:GND") (at 58.42 59.69 0) (unit 1)
     (in_bom yes) (on_board yes)
-    (property "Reference" "#PWR?" (id 0) (at 58.42 66.04 0)
+    (property "Reference" "#PWR0102" (id 0) (at 58.42 66.04 0)
       (effects (font (size 1.27 1.27)) hide)
     )
@@
   (symbol (lib_id "power:GND") (at 100.33 59.69 0) (unit 1)
     (in_bom yes) (on_board yes)
-    (property "Reference" "#PWR?" (id 0) (at 100.33 66.04 0)
+    (property "Reference" "#PWR0111" (id 0) (at 100.33 66.04 0)
       (effects (font (size 1.27 1.27)) hide)
     )
@@
   (symbol (lib_id "power:GND") (at 104.648 59.69 0) (unit 1)
     (in_bom yes) (on_board yes)
-    (property "Reference" "#PWR?" (id 0) (at 104.648 66.04 0)
+    (property "Reference" "#PWR0112" (id 0) (at 104.648 66.04 0)
       (effects (font (size 1.27 1.27)) hide)
     )
@@
   (symbol (lib_id "power:GND") (at 118.11 59.69 0) (unit 1)
     (in_bom yes) (on_board yes)
-    (property "Reference" "#PWR?" (id 0) (at 118.11 66.04 0)
+    (property "Reference" "#PWR0114" (id 0) (at 118.11 66.04 0)
       (effects (font (size 1.27 1.27)) hide)
     )
@@
   (symbol (lib_id "power:GND") (at 128.27 59.69 0) (unit 1)
     (in_bom yes) (on_board yes)
-    (property "Reference" "#PWR?" (id 0) (at 128.27 66.04 0)
+    (property "Reference" "#PWR0113" (id 0) (at 128.27 66.04 0)
       (effects (font (size 1.27 1.27)) hide)
     )
@@
   (symbol (lib_id "power:GND") (at 138.43 59.69 0) (unit 1)
     (in_bom yes) (on_board yes)
-    (property "Reference" "#PWR?" (id 0) (at 138.43 66.04 0)
+    (property "Reference" "#PWR0115" (id 0) (at 138.43 66.04 0)
       (effects (font (size 1.27 1.27)) hide)
     )
@@
   (symbol (lib_id "power:GND") (at 148.59 59.69 0) (unit 1)
     (in_bom yes) (on_board yes)
-    (property "Reference" "#PWR?" (id 0) (at 148.59 66.04 0)
+    (property "Reference" "#PWR0110" (id 0) (at 148.59 66.04 0)
       (effects (font (size 1.27 1.27)) hide)
     )
@@
   (symbol (lib_id "power:GND") (at 186.69 92.71 0) (unit 1)
     (in_bom yes) (on_board yes)
-    (property "Reference" "#PWR?" (id 0) (at 186.69 99.06 0)
+    (property "Reference" "#PWR0103" (id 0) (at 186.69 99.06 0)
       (effects (font (size 1.27 1.27)) hide)
     )
@@
   (symbol (lib_id "power:GND") (at 238.76 125.73 0) (unit 1)
     (in_bom yes) (on_board yes)
-    (property "Reference" "#PWR?" (id 0) (at 238.76 132.08 0)
+    (property "Reference" "#PWR0106" (id 0) (at 238.76 132.08 0)
       (effects (font (size 1.27 1.27)) hide)
     )
@@
   (symbol (lib_id "power:GND") (at 242.57 125.73 0) (unit 1)
     (in_bom yes) (on_board yes)
-    (property "Reference" "#PWR?" (id 0) (at 242.57 132.08 0)
+    (property "Reference" "#PWR0107" (id 0) (at 242.57 132.08 0)
       (effects (font (size 1.27 1.27)) hide)
     )
@@
   (symbol (lib_id "power:GND") (at 243.84 36.83 0) (unit 1)
     (in_bom yes) (on_board yes)
-    (property "Reference" "#PWR?" (id 0) (at 243.84 43.18 0)
+    (property "Reference" "#PWR0104" (id 0) (at 243.84 43.18 0)
       (effects (font (size 1.27 1.27)) hide)
     )
@@
   (symbol (lib_id "power:GND") (at 248.92 125.73 0) (unit 1)
     (in_bom yes) (on_board yes)
-    (property "Reference" "#PWR?" (id 0) (at 248.92 132.08 0)
+    (property "Reference" "#PWR0105" (id 0) (at 248.92 132.08 0)
       (effects (font (size 1.27 1.27)) hide)
     )
@@
   (symbol (lib_id "power:GND") (at 275.59 27.94 0) (unit 1)
     (in_bom yes) (on_board yes)
-    (property "Reference" "#PWR?" (id 0) (at 275.59 34.29 0)
+    (property "Reference" "#PWR0108" (id 0) (at 275.59 34.29 0)
       (effects (font (size 1.27 1.27)) hide)
     )
@@
   (symbol (lib_id "power:GND") (at 276.86 104.14 0) (unit 1)
     (in_bom yes) (on_board yes)
-    (property "Reference" "#PWR?" (id 0) (at 276.86 110.49 0)
+    (property "Reference" "#PWR0109" (id 0) (at 276.86 110.49 0)
       (effects (font (size 1.27 1.27)) hide)
     )
@@
   (symbol (lib_id "Device:R") (at 96.52 52.07 90) (unit 1)
     (in_bom yes) (on_board yes)
-    (property "Reference" "R?" (id 0) (at 100.33 48.26 90)
+    (property "Reference" "R1" (id 0) (at 100.33 48.26 90)
       (effects (font (size 1.27 1.27)) (justify left))
     )
@@
       (effects (font (size 1.27 1.27)) (justify left))
     )
-    (property "Footprint" "Resistor_SMD:R_0805_2012Metric" (id 2) (at 96.52 53.848 90)
+    (property "Footprint" "Resistor_SMD:R_0603_1608Metric" (id 2) (at 96.52 53.848 90)
       (effects (font (size 1.27 1.27)) hide)
     )
@@
   (symbol (lib_id "Device:R") (at 238.76 118.11 0) (unit 1)
     (in_bom yes) (on_board yes) (fields_autoplaced)
-    (property "Reference" "R?" (id 0) (at 241.3 117.4749 0)
+    (property "Reference" "R2" (id 0) (at 241.3 117.4749 0)
       (effects (font (size 1.27 1.27)) (justify left))
     )
@@
   (symbol (lib_id "Device:R") (at 242.57 118.11 0) (unit 1)
     (in_bom yes) (on_board yes) (fields_autoplaced)
-    (property "Reference" "R?" (id 0) (at 245.11 117.4749 0)
+    (property "Reference" "R3" (id 0) (at 245.11 117.4749 0)
       (effects (font (size 1.27 1.27)) (justify left))
     )
@@
   (symbol (lib_id "Device:C") (at 46.99 54.61 0) (unit 1)
     (in_bom yes) (on_board yes)
-    (property "Reference" "C?" (id 0) (at 49.911 53.4416 0)
+    (property "Reference" "C1" (id 0) (at 49.911 53.4416 0)
       (effects (font (size 1.27 1.27)) (justify left))
     )
@@
   (symbol (lib_id "Device:CP") (at 104.648 55.88 0) (unit 1)
     (in_bom yes) (on_board yes)
-    (property "Reference" "C?" (id 0) (at 107.6452 54.737 0)
+    (property "Reference" "C2" (id 0) (at 107.6452 54.737 0)
       (effects (font (size 1.27 1.27)) (justify left))
     )
@@
   (symbol (lib_id "Device:C") (at 118.11 55.88 0) (unit 1)
     (in_bom yes) (on_board yes)
-    (property "Reference" "C?" (id 0) (at 121.031 54.7116 0)
+    (property "Reference" "C3" (id 0) (at 121.031 54.7116 0)
       (effects (font (size 1.27 1.27)) (justify left))
     )
@@
   (symbol (lib_id "Device:C") (at 128.27 55.88 0) (unit 1)
     (in_bom yes) (on_board yes)
-    (property "Reference" "C?" (id 0) (at 131.191 54.7116 0)
+    (property "Reference" "C4" (id 0) (at 131.191 54.7116 0)
       (effects (font (size 1.27 1.27)) (justify left))
     )
@@
   (symbol (lib_id "Device:C") (at 138.43 55.88 0) (unit 1)
     (in_bom yes) (on_board yes)
-    (property "Reference" "C?" (id 0) (at 141.351 54.7116 0)
+    (property "Reference" "C5" (id 0) (at 141.351 54.7116 0)
       (effects (font (size 1.27 1.27)) (justify left))
     )
@@
   (symbol (lib_id "Device:C") (at 148.59 55.88 0) (unit 1)
     (in_bom yes) (on_board yes)
-    (property "Reference" "C?" (id 0) (at 151.511 54.7116 0)
+    (property "Reference" "C6" (id 0) (at 151.511 54.7116 0)
       (effects (font (size 1.27 1.27)) (justify left))
     )
@@
   (symbol (lib_id "CM4IO:AP2553W6") (at 77.47 52.07 0) (unit 1)
     (in_bom yes) (on_board yes)
-    (property "Reference" "U?" (id 0) (at 76.835 42.799 0))
+    (property "Reference" "U1" (id 0) (at 76.835 42.799 0))
     (property "Value" "AP22653W6" (id 1) (at 76.835 45.1104 0))
     (property "Footprint" "Package_TO_SOT_SMD:SOT-23-6" (id 2) (at 81.28 58.42 0)
@@
   (symbol (lib_id "CM4IO:TPD4EUSB30") (at 186.69 80.01 0) (unit 1)
     (in_bom yes) (on_board yes)
-    (property "Reference" "U?" (id 0) (at 186.69 68.1482 0))
+    (property "Reference" "U2" (id 0) (at 186.69 68.1482 0))
     (property "Value" "TPD4EUSB30" (id 1) (at 186.69 70.4596 0))
     (property "Footprint" "Package_SON:USON-10_2.5x1.0mm_P0.5mm" (id 2) (at 162.56 90.17 0)
@@
   (symbol (lib_id "CM4IO:USB_A") (at 262.89 50.8 0) (unit 1)
     (in_bom yes) (on_board yes) (fields_autoplaced)
-    (property "Reference" "J?" (id 0) (at 261.62 20.32 0))
+    (property "Reference" "J1" (id 0) (at 261.62 20.32 0))
     (property "Value" "USB_A" (id 1) (at 261.62 22.86 0))
     (property "Footprint" "cm4crypto:OnShore_USB-A1HSB6" (id 2) (at 264.16 30.48 0)
@@
   (symbol (lib_id "cm4crypto:USB_C") (at 264.16 127 0) (unit 1)
     (in_bom yes) (on_board yes) (fields_autoplaced)
-    (property "Reference" "J?" (id 0) (at 262.89 96.52 0))
+    (property "Reference" "J2" (id 0) (at 262.89 96.52 0))
     (property "Value" "USB_C" (id 1) (at 262.89 99.06 0))
     (property "Footprint" "cm4crypto:USB4105-GF-A" (id 2) (at 265.43 106.68 0)

Commit message: tweak mezzanine
almost ready to order
Parts:
- C1, C3, C4, C5, C6: footprint Capacitor_SMD:C_0805_2012Metric -> Capacitor_SMD:C_0603_1608Metric
- J1: footprint cm4crypto:OnShore_USB-A1HSB6 -> cm4crypto:AU-Y1006
Connections:
- net +5v is gone; now on net VBUS: C1.1, U1.1 (IN), U1.3 (EN)
Changed lines of the file:
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@@
     (effects (font (size 1.27 1.27)) (justify left bottom))
   )
-  (label "USB2_HOST_VBUS" (at 105.41 49.53 0)
+  (label "USB2_HOST_VBUS" (at 151.13 49.53 0)
     (effects (font (size 1.27 1.27)) (justify left bottom))
   )
@@
     (effects (font (size 1.27 1.27)) (justify right bottom))
   )
+  (global_label "+5v" (shape output) (at 229.87 102.87 180) (fields_autoplaced)
+    (effects (font (size 1.27 1.27)) (justify right))
+    (property "Intersheet References" "${INTERSHEET_REFS}" (id 0) (at 223.7074 102.7906 0)
+      (effects (font (size 1.27 1.27)) (justify right) hide)
+    )
+  )
   (hierarchical_label "+5v" (shape input) (at 60.96 22.86 180)
     (effects (font (size 1.27 1.27)) (justify right))
@@
     (effects (font (size 1.27 1.27)) (justify right))
   )
-  (hierarchical_label "USB2_DEV_VBUS" (shape output) (at 229.87 102.87 180)
-    (effects (font (size 1.27 1.27)) (justify right))
-  )
   (hierarchical_label "USB2_DEV_N" (shape bidirectional) (at 229.87 105.41 180)
     (effects (font (size 1.27 1.27)) (justify right))
@@
   (symbol (lib_id "power:GND") (at 46.99 58.42 0) (unit 1)
     (in_bom yes) (on_board yes)
-    (property "Reference" "#PWR0101" (id 0) (at 46.99 64.77 0)
+    (property "Reference" "#PWR033" (id 0) (at 46.99 64.77 0)
       (effects (font (size 1.27 1.27)) hide)
     )
@@
   (symbol (lib_id "power:GND") (at 58.42 59.69 0) (unit 1)
     (in_bom yes) (on_board yes)
-    (property "Reference" "#PWR0102" (id 0) (at 58.42 66.04 0)
+    (property "Reference" "#PWR034" (id 0) (at 58.42 66.04 0)
       (effects (font (size 1.27 1.27)) hide)
     )
@@
   (symbol (lib_id "power:GND") (at 100.33 59.69 0) (unit 1)
     (in_bom yes) (on_board yes)
-    (property "Reference" "#PWR0111" (id 0) (at 100.33 66.04 0)
+    (property "Reference" "#PWR035" (id 0) (at 100.33 66.04 0)
       (effects (font (size 1.27 1.27)) hide)
     )
@@
   (symbol (lib_id "power:GND") (at 104.648 59.69 0) (unit 1)
     (in_bom yes) (on_board yes)
-    (property "Reference" "#PWR0112" (id 0) (at 104.648 66.04 0)
+    (property "Reference" "#PWR036" (id 0) (at 104.648 66.04 0)
       (effects (font (size 1.27 1.27)) hide)
     )
@@
   (symbol (lib_id "power:GND") (at 118.11 59.69 0) (unit 1)
     (in_bom yes) (on_board yes)
-    (property "Reference" "#PWR0114" (id 0) (at 118.11 66.04 0)
+    (property "Reference" "#PWR037" (id 0) (at 118.11 66.04 0)
       (effects (font (size 1.27 1.27)) hide)
     )
@@
   (symbol (lib_id "power:GND") (at 128.27 59.69 0) (unit 1)
     (in_bom yes) (on_board yes)
-    (property "Reference" "#PWR0113" (id 0) (at 128.27 66.04 0)
+    (property "Reference" "#PWR038" (id 0) (at 128.27 66.04 0)
       (effects (font (size 1.27 1.27)) hide)
     )
@@
   (symbol (lib_id "power:GND") (at 138.43 59.69 0) (unit 1)
     (in_bom yes) (on_board yes)
-    (property "Reference" "#PWR0115" (id 0) (at 138.43 66.04 0)
+    (property "Reference" "#PWR039" (id 0) (at 138.43 66.04 0)
       (effects (font (size 1.27 1.27)) hide)
     )
@@
   (symbol (lib_id "power:GND") (at 148.59 59.69 0) (unit 1)
     (in_bom yes) (on_board yes)
-    (property "Reference" "#PWR0110" (id 0) (at 148.59 66.04 0)
+    (property "Reference" "#PWR040" (id 0) (at 148.59 66.04 0)
       (effects (font (size 1.27 1.27)) hide)
     )
@@
   (symbol (lib_id "power:GND") (at 186.69 92.71 0) (unit 1)
     (in_bom yes) (on_board yes)
-    (property "Reference" "#PWR0103" (id 0) (at 186.69 99.06 0)
+    (property "Reference" "#PWR041" (id 0) (at 186.69 99.06 0)
       (effects (font (size 1.27 1.27)) hide)
     )
@@
   (symbol (lib_id "power:GND") (at 238.76 125.73 0) (unit 1)
     (in_bom yes) (on_board yes)
-    (property "Reference" "#PWR0106" (id 0) (at 238.76 132.08 0)
+    (property "Reference" "#PWR043" (id 0) (at 238.76 132.08 0)
       (effects (font (size 1.27 1.27)) hide)
     )
@@
   (symbol (lib_id "power:GND") (at 242.57 125.73 0) (unit 1)
     (in_bom yes) (on_board yes)
-    (property "Reference" "#PWR0107" (id 0) (at 242.57 132.08 0)
+    (property "Reference" "#PWR044" (id 0) (at 242.57 132.08 0)
       (effects (font (size 1.27 1.27)) hide)
     )
@@
   (symbol (lib_id "power:GND") (at 243.84 36.83 0) (unit 1)
     (in_bom yes) (on_board yes)
-    (property "Reference" "#PWR0104" (id 0) (at 243.84 43.18 0)
+    (property "Reference" "#PWR032" (id 0) (at 243.84 43.18 0)
       (effects (font (size 1.27 1.27)) hide)
     )
@@
   (symbol (lib_id "power:GND") (at 248.92 125.73 0) (unit 1)
     (in_bom yes) (on_board yes)
-    (property "Reference" "#PWR0105" (id 0) (at 248.92 132.08 0)
+    (property "Reference" "#PWR045" (id 0) (at 248.92 132.08 0)
       (effects (font (size 1.27 1.27)) hide)
     )
@@
   (symbol (lib_id "power:GND") (at 275.59 27.94 0) (unit 1)
     (in_bom yes) (on_board yes)
-    (property "Reference" "#PWR0108" (id 0) (at 275.59 34.29 0)
+    (property "Reference" "#PWR031" (id 0) (at 275.59 34.29 0)
       (effects (font (size 1.27 1.27)) hide)
     )
@@
   (symbol (lib_id "power:GND") (at 276.86 104.14 0) (unit 1)
     (in_bom yes) (on_board yes)
-    (property "Reference" "#PWR0109" (id 0) (at 276.86 110.49 0)
+    (property "Reference" "#PWR042" (id 0) (at 276.86 110.49 0)
       (effects (font (size 1.27 1.27)) hide)
     )
@@
       (effects (font (size 1.27 1.27)) (justify left))
     )
-    (property "Footprint" "Capacitor_SMD:C_0805_2012Metric" (id 2) (at 47.9552 58.42 0)
+    (property "Footprint" "Capacitor_SMD:C_0603_1608Metric" (id 2) (at 47.9552 58.42 0)
       (effects (font (size 1.27 1.27)) hide)
     )
@@
       (effects (font (size 1.27 1.27)) (justify left))
     )
-    (property "Footprint" "Capacitor_SMD:C_0805_2012Metric" (id 2) (at 119.0752 59.69 0)
+    (property "Footprint" "Capacitor_SMD:C_0603_1608Metric" (id 2) (at 119.0752 59.69 0)
       (effects (font (size 1.27 1.27)) hide)
     )
@@
       (effects (font (size 1.27 1.27)) (justify left))
     )
-    (property "Footprint" "Capacitor_SMD:C_0805_2012Metric" (id 2) (at 129.2352 59.69 0)
+    (property "Footprint" "Capacitor_SMD:C_0603_1608Metric" (id 2) (at 129.2352 59.69 0)
       (effects (font (size 1.27 1.27)) hide)
     )
@@
       (effects (font (size 1.27 1.27)) (justify left))
     )
-    (property "Footprint" "Capacitor_SMD:C_0805_2012Metric" (id 2) (at 139.3952 59.69 0)
+    (property "Footprint" "Capacitor_SMD:C_0603_1608Metric" (id 2) (at 139.3952 59.69 0)
       (effects (font (size 1.27 1.27)) hide)
     )
@@
       (effects (font (size 1.27 1.27)) (justify left))
     )
-    (property "Footprint" "Capacitor_SMD:C_0805_2012Metric" (id 2) (at 149.5552 59.69 0)
+    (property "Footprint" "Capacitor_SMD:C_0603_1608Metric" (id 2) (at 149.5552 59.69 0)
       (effects (font (size 1.27 1.27)) hide)
     )
@@
     (property "Reference" "J1" (id 0) (at 261.62 20.32 0))
     (property "Value" "USB_A" (id 1) (at 261.62 22.86 0))
-    (property "Footprint" "cm4crypto:OnShore_USB-A1HSB6" (id 2) (at 264.16 30.48 0)
-      (effects (font (size 1.27 1.27)) hide)
-    )
+    (property "Footprint" "cm4crypto:AU-Y1006" (id 2) (at 264.16 30.48 0)
+      (effects (font (size 1.27 1.27)) hide)
+    )

Commit message: update USB-A host capacitor footprint
Parts:
- C2: footprint Capacitor_Tantalum_SMD:CP_EIA-7343-31_Kemet-D -> Capacitor_SMD:C_0805_2012Metric_Pad1.18x1.45mm_HandSolder
Changed lines of the file:
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@@
       (effects (font (size 1.27 1.27)) (justify left))
     )
-    (property "Footprint" "Capacitor_Tantalum_SMD:CP_EIA-7343-31_Kemet-D" (id 2) (at 105.6132 59.69 0)
+    (property "Footprint" "Capacitor_SMD:C_0805_2012Metric_Pad1.18x1.45mm_HandSolder" (id 2) (at 105.6132 59.69 0)
       (effects (font (size 1.27 1.27)) hide)
     )
