File: hardware/lobby/sheets/jumpers.kicad_sch (KiCad schematic)
At the start: 9 parts

Commit message: start routing mezzanine
making a progress capture before trying to cram a lot of signals onto just one hirose connector...
Parts:
- removed R?: 0R, Resistor_SMD:R_0805_2012Metric_Pad1.15x1.40mm_HandSolder, symbol Device:R
- removed R?: nf, Resistor_SMD:R_0805_2012Metric_Pad1.15x1.40mm_HandSolder, symbol Device:R
- added JP5: Jumper_2_Bridged, Jumper:SolderJumper-2_P1.3mm_Bridged_Pad1.0x1.5mm, symbol Jumper:Jumper_2_Bridged
- added JP6: SolderJumper_2_Open, Jumper:SolderJumper-2_P1.3mm_Open_TrianglePad1.0x1.5mm, symbol Jumper:SolderJumper_2_Open
- JP1, JP2, JP3, JP4: renamed from JP?; footprint (none) -> Jumper:SolderJumper-2_P1.3mm_Open_TrianglePad1.0x1.5mm
- SW1: renamed from SW?; footprint (none) -> cm4crypto:EVQ-P7C01P
- SW2: renamed from SW?; footprint (none) -> cm4crypto:cus-12b
- gave numbers to parts that had none: 1
Connections:
- net +1.8v: now also JP6.1 (A)
- net +3.3v: now also JP5.1 (A)
- net GPIO_VREF: now also JP5.2 (B), JP6.2 (B)

Commit message: sheet refs relative, copied escalator pinout to lobby
Parts:
- renumbered JP5 to JP?, JP2 to JP?, JP6 to JP?, JP3 to JP?, JP1 to JP?, JP4 to JP?, R6 to R?, SW1 to SW?, SW2 to SW?
Changed lines of the file:
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@@
   (symbol (lib_id "power:GND") (at 39.37 133.35 0) (unit 1)
     (in_bom yes) (on_board yes) (fields_autoplaced)
-    (property "Reference" "#PWR059" (id 0) (at 39.37 139.7 0)
+    (property "Reference" "#PWR?" (id 0) (at 39.37 139.7 0)
       (effects (font (size 1.27 1.27)) hide)
     )
@@
   (symbol (lib_id "power:GND") (at 45.72 67.31 0) (unit 1)
     (in_bom yes) (on_board yes)
-    (property "Reference" "#PWR056" (id 0) (at 45.72 73.66 0)
+    (property "Reference" "#PWR?" (id 0) (at 45.72 73.66 0)
       (effects (font (size 1.27 1.27)) hide)
     )
@@
   (symbol (lib_id "power:GND") (at 45.72 85.09 0) (unit 1)
     (in_bom yes) (on_board yes)
-    (property "Reference" "#PWR057" (id 0) (at 45.72 91.44 0)
+    (property "Reference" "#PWR?" (id 0) (at 45.72 91.44 0)
       (effects (font (size 1.27 1.27)) hide)
     )
@@
   (symbol (lib_id "power:GND") (at 45.72 99.06 0) (unit 1)
     (in_bom yes) (on_board yes)
-    (property "Reference" "#PWR058" (id 0) (at 45.72 105.41 0)
+    (property "Reference" "#PWR?" (id 0) (at 45.72 105.41 0)
       (effects (font (size 1.27 1.27)) hide)
     )
@@
   (symbol (lib_id "power:GND") (at 46.99 36.83 0) (unit 1)
     (in_bom yes) (on_board yes)
-    (property "Reference" "#PWR055" (id 0) (at 46.99 43.18 0)
+    (property "Reference" "#PWR?" (id 0) (at 46.99 43.18 0)
       (effects (font (size 1.27 1.27)) hide)
     )
@@
   (symbol (lib_id "Jumper:Jumper_2_Bridged") (at 39.37 153.67 0) (unit 1)
     (in_bom yes) (on_board yes)
-    (property "Reference" "JP5" (id 0) (at 39.37 148.59 0))
+    (property "Reference" "JP?" (id 0) (at 39.37 148.59 0))
     (property "Value" "Jumper_2_Bridged" (id 1) (at 39.37 151.13 0))
     (property "Footprint" "Jumper:SolderJumper-2_P1.3mm_Bridged_Pad1.0x1.5mm" (id 2) (at 39.37 153.67 0)
@@
   (symbol (lib_id "Jumper:SolderJumper_2_Open") (at 40.64 34.29 0) (unit 1)
     (in_bom yes) (on_board yes) (fields_autoplaced)
-    (property "Reference" "JP1" (id 0) (at 40.64 29.21 0))
+    (property "Reference" "JP?" (id 0) (at 40.64 29.21 0))
     (property "Value" "SolderJumper_2_Open" (id 1) (at 40.64 31.75 0))
     (property "Footprint" "Jumper:SolderJumper-2_P1.3mm_Open_TrianglePad1.0x1.5mm" (id 2) (at 40.64 34.29 0)
@@
   (symbol (lib_id "Jumper:SolderJumper_2_Open") (at 40.64 66.04 0) (unit 1)
     (in_bom yes) (on_board yes) (fields_autoplaced)
-    (property "Reference" "JP2" (id 0) (at 40.64 60.96 0))
+    (property "Reference" "JP?" (id 0) (at 40.64 60.96 0))
     (property "Value" "SolderJumper_2_Open" (id 1) (at 40.64 63.5 0))
     (property "Footprint" "Jumper:SolderJumper-2_P1.3mm_Open_TrianglePad1.0x1.5mm" (id 2) (at 40.64 66.04 0)
@@
   (symbol (lib_id "Jumper:SolderJumper_2_Open") (at 40.64 83.82 0) (unit 1)
     (in_bom yes) (on_board yes) (fields_autoplaced)
-    (property "Reference" "JP3" (id 0) (at 40.64 78.74 0))
+    (property "Reference" "JP?" (id 0) (at 40.64 78.74 0))
     (property "Value" "SolderJumper_2_Open" (id 1) (at 40.64 81.28 0))
     (property "Footprint" "Jumper:SolderJumper-2_P1.3mm_Open_TrianglePad1.0x1.5mm" (id 2) (at 40.64 83.82 0)
@@
   (symbol (lib_id "Jumper:SolderJumper_2_Open") (at 40.64 97.79 0) (unit 1)
     (in_bom yes) (on_board yes)
-    (property "Reference" "JP4" (id 0) (at 40.64 92.71 0))
+    (property "Reference" "JP?" (id 0) (at 40.64 92.71 0))
     (property "Value" "SolderJumper_2_Open" (id 1) (at 40.64 95.25 0))
     (property "Footprint" "Jumper:SolderJumper-2_P1.3mm_Open_TrianglePad1.0x1.5mm" (id 2) (at 40.64 97.79 0)
@@
   (symbol (lib_id "Jumper:SolderJumper_2_Open") (at 41.91 157.48 0) (unit 1)
     (in_bom yes) (on_board yes)
-    (property "Reference" "JP6" (id 0) (at 41.91 152.4 0))
+    (property "Reference" "JP?" (id 0) (at 41.91 152.4 0))
     (property "Value" "SolderJumper_2_Open" (id 1) (at 41.91 154.94 0))
     (property "Footprint" "Jumper:SolderJumper-2_P1.3mm_Open_TrianglePad1.0x1.5mm" (id 2) (at 41.91 157.48 0)
@@
   (symbol (lib_id "Device:R") (at 39.37 128.27 0) (unit 1)
     (in_bom yes) (on_board yes) (fields_autoplaced)
-    (property "Reference" "R6" (id 0) (at 41.91 127.6349 0)
+    (property "Reference" "R?" (id 0) (at 41.91 127.6349 0)
       (effects (font (size 1.27 1.27)) (justify left))
     )
@@
   (symbol (lib_id "Switch:SW_SPST") (at 33.02 123.19 0) (unit 1)
     (in_bom yes) (on_board yes) (fields_autoplaced)
-    (property "Reference" "SW2" (id 0) (at 33.02 118.11 0))
+    (property "Reference" "SW?" (id 0) (at 33.02 118.11 0))
     (property "Value" "SW_SPST" (id 1) (at 33.02 120.65 0))
     (property "Footprint" "cm4crypto:cus-12b" (id 2) (at 33.02 123.19 0)
@@
   (symbol (lib_id "Switch:SW_Push") (at 40.64 30.48 0) (unit 1)
     (in_bom yes) (on_board yes) (fields_autoplaced)
-    (property "Reference" "SW1" (id 0) (at 40.64 24.13 0))
+    (property "Reference" "SW?" (id 0) (at 40.64 24.13 0))
     (property "Value" "SW_Push" (id 1) (at 40.64 26.67 0))
     (property "Footprint" "cm4crypto:EVQ-P7C01P" (id 2) (at 40.64 25.4 0)

Commit message: work abroad
did some light planning for the lobby board while on vacation. now ready for final placement + routing
Parts:
- gave numbers to parts that had none: 9
Changed lines of the file:
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@@
   (symbol (lib_id "power:GND") (at 39.37 133.35 0) (unit 1)
     (in_bom yes) (on_board yes) (fields_autoplaced)
-    (property "Reference" "#PWR?" (id 0) (at 39.37 139.7 0)
+    (property "Reference" "#PWR058" (id 0) (at 39.37 139.7 0)
       (effects (font (size 1.27 1.27)) hide)
     )
@@
   (symbol (lib_id "power:GND") (at 45.72 67.31 0) (unit 1)
     (in_bom yes) (on_board yes)
-    (property "Reference" "#PWR?" (id 0) (at 45.72 73.66 0)
+    (property "Reference" "#PWR059" (id 0) (at 45.72 73.66 0)
       (effects (font (size 1.27 1.27)) hide)
     )
@@
   (symbol (lib_id "power:GND") (at 45.72 85.09 0) (unit 1)
     (in_bom yes) (on_board yes)
-    (property "Reference" "#PWR?" (id 0) (at 45.72 91.44 0)
+    (property "Reference" "#PWR060" (id 0) (at 45.72 91.44 0)
       (effects (font (size 1.27 1.27)) hide)
     )
@@
   (symbol (lib_id "power:GND") (at 45.72 99.06 0) (unit 1)
     (in_bom yes) (on_board yes)
-    (property "Reference" "#PWR?" (id 0) (at 45.72 105.41 0)
+    (property "Reference" "#PWR061" (id 0) (at 45.72 105.41 0)
       (effects (font (size 1.27 1.27)) hide)
     )
@@
   (symbol (lib_id "power:GND") (at 46.99 36.83 0) (unit 1)
     (in_bom yes) (on_board yes)
-    (property "Reference" "#PWR?" (id 0) (at 46.99 43.18 0)
+    (property "Reference" "#PWR062" (id 0) (at 46.99 43.18 0)
       (effects (font (size 1.27 1.27)) hide)
     )
@@
   (symbol (lib_id "Jumper:Jumper_2_Bridged") (at 39.37 153.67 0) (unit 1)
     (in_bom yes) (on_board yes)
-    (property "Reference" "JP?" (id 0) (at 39.37 148.59 0))
+    (property "Reference" "JP1" (id 0) (at 39.37 148.59 0))
     (property "Value" "Jumper_2_Bridged" (id 1) (at 39.37 151.13 0))
     (property "Footprint" "Jumper:SolderJumper-2_P1.3mm_Bridged_Pad1.0x1.5mm" (id 2) (at 39.37 153.67 0)
@@
   (symbol (lib_id "Jumper:SolderJumper_2_Open") (at 40.64 34.29 0) (unit 1)
     (in_bom yes) (on_board yes) (fields_autoplaced)
-    (property "Reference" "JP?" (id 0) (at 40.64 29.21 0))
+    (property "Reference" "JP2" (id 0) (at 40.64 29.21 0))
     (property "Value" "SolderJumper_2_Open" (id 1) (at 40.64 31.75 0))
     (property "Footprint" "Jumper:SolderJumper-2_P1.3mm_Open_TrianglePad1.0x1.5mm" (id 2) (at 40.64 34.29 0)
@@
   (symbol (lib_id "Jumper:SolderJumper_2_Open") (at 40.64 66.04 0) (unit 1)
     (in_bom yes) (on_board yes) (fields_autoplaced)
-    (property "Reference" "JP?" (id 0) (at 40.64 60.96 0))
+    (property "Reference" "JP3" (id 0) (at 40.64 60.96 0))
     (property "Value" "SolderJumper_2_Open" (id 1) (at 40.64 63.5 0))
     (property "Footprint" "Jumper:SolderJumper-2_P1.3mm_Open_TrianglePad1.0x1.5mm" (id 2) (at 40.64 66.04 0)
@@
   (symbol (lib_id "Jumper:SolderJumper_2_Open") (at 40.64 83.82 0) (unit 1)
     (in_bom yes) (on_board yes) (fields_autoplaced)
-    (property "Reference" "JP?" (id 0) (at 40.64 78.74 0))
+    (property "Reference" "JP4" (id 0) (at 40.64 78.74 0))
     (property "Value" "SolderJumper_2_Open" (id 1) (at 40.64 81.28 0))
     (property "Footprint" "Jumper:SolderJumper-2_P1.3mm_Open_TrianglePad1.0x1.5mm" (id 2) (at 40.64 83.82 0)
@@
   (symbol (lib_id "Jumper:SolderJumper_2_Open") (at 40.64 97.79 0) (unit 1)
     (in_bom yes) (on_board yes)
-    (property "Reference" "JP?" (id 0) (at 40.64 92.71 0))
+    (property "Reference" "JP5" (id 0) (at 40.64 92.71 0))
     (property "Value" "SolderJumper_2_Open" (id 1) (at 40.64 95.25 0))
     (property "Footprint" "Jumper:SolderJumper-2_P1.3mm_Open_TrianglePad1.0x1.5mm" (id 2) (at 40.64 97.79 0)
@@
   (symbol (lib_id "Jumper:SolderJumper_2_Open") (at 41.91 157.48 0) (unit 1)
     (in_bom yes) (on_board yes)
-    (property "Reference" "JP?" (id 0) (at 41.91 152.4 0))
+    (property "Reference" "JP6" (id 0) (at 41.91 152.4 0))
     (property "Value" "SolderJumper_2_Open" (id 1) (at 41.91 154.94 0))
     (property "Footprint" "Jumper:SolderJumper-2_P1.3mm_Open_TrianglePad1.0x1.5mm" (id 2) (at 41.91 157.48 0)
@@
   (symbol (lib_id "Device:R") (at 39.37 128.27 0) (unit 1)
     (in_bom yes) (on_board yes) (fields_autoplaced)
-    (property "Reference" "R?" (id 0) (at 41.91 127.6349 0)
+    (property "Reference" "R6" (id 0) (at 41.91 127.6349 0)
       (effects (font (size 1.27 1.27)) (justify left))
     )
@@
   (symbol (lib_id "Switch:SW_SPST") (at 33.02 123.19 0) (unit 1)
     (in_bom yes) (on_board yes) (fields_autoplaced)
-    (property "Reference" "SW?" (id 0) (at 33.02 118.11 0))
+    (property "Reference" "SW1" (id 0) (at 33.02 118.11 0))
     (property "Value" "SW_SPST" (id 1) (at 33.02 120.65 0))
     (property "Footprint" "cm4crypto:cus-12b" (id 2) (at 33.02 123.19 0)
@@
   (symbol (lib_id "Switch:SW_Push") (at 40.64 30.48 0) (unit 1)
     (in_bom yes) (on_board yes) (fields_autoplaced)
-    (property "Reference" "SW?" (id 0) (at 40.64 24.13 0))
+    (property "Reference" "SW2" (id 0) (at 40.64 24.13 0))
     (property "Value" "SW_Push" (id 1) (at 40.64 26.67 0))
     (property "Footprint" "cm4crypto:EVQ-P7C01P" (id 2) (at 40.64 25.4 0)

Commit message: place lobby components
Parts:
- removed JP1: Jumper_2_Bridged, Jumper:SolderJumper-2_P1.3mm_Bridged_Pad1.0x1.5mm, symbol Jumper:Jumper_2_Bridged
- removed JP6: SolderJumper_2_Open, Jumper:SolderJumper-2_P1.3mm_Open_TrianglePad1.0x1.5mm, symbol Jumper:SolderJumper_2_Open
- added JP5: Jumper_3_Bridged12, Jumper:SolderJumper-3_P1.3mm_Bridged12_RoundedPad1.0x1.5mm, symbol Jumper:Jumper_3_Bridged12
- JP1: renamed from JP2; footprint Jumper:SolderJumper-2_P1.3mm_Open_TrianglePad1.0x1.5mm -> Jumper:SolderJumper-2_P1.3mm_Open_RoundedPad1.0x1.5mm
- JP2: renamed from JP3; footprint Jumper:SolderJumper-2_P1.3mm_Open_TrianglePad1.0x1.5mm -> Jumper:SolderJumper-2_P1.3mm_Open_RoundedPad1.0x1.5mm
- JP3: renamed from JP4; footprint Jumper:SolderJumper-2_P1.3mm_Open_TrianglePad1.0x1.5mm -> Jumper:SolderJumper-2_P1.3mm_Open_RoundedPad1.0x1.5mm
- JP4: renamed from JP5; footprint Jumper:SolderJumper-2_P1.3mm_Open_TrianglePad1.0x1.5mm -> Jumper:SolderJumper-2_P1.3mm_Open_RoundedPad1.0x1.5mm
- renumbered SW2 to SW1, SW1 to SW2
Connections:
- net +1.8v: now also JP5.3 (B)
- net +3.3v: now also JP5.1 (A)
- net GPIO_VREF: now also JP5.2 (C)
Changed lines of the file:
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@@
   (junction (at 39.37 123.19) (diameter 0.9144) (color 0 0 0 0))
   (junction (at 46.99 34.29) (diameter 1.016) (color 0 0 0 0))
-  (junction (at 46.99 153.67) (diameter 0.9144) (color 0 0 0 0))
   (wire (pts (xy 22.86 30.48) (xy 34.29 30.48))
     (stroke (width 0) (type solid) (color 0 0 0 0))
   )
-  (wire (pts (xy 25.4 153.67) (xy 34.29 153.67))
-    (stroke (width 0) (type solid) (color 0 0 0 0))
-  )
-  (wire (pts (xy 25.4 157.48) (xy 38.1 157.48))
-    (stroke (width 0) (type solid) (color 0 0 0 0))
-  )
   (wire (pts (xy 26.67 66.04) (xy 36.83 66.04))
     (stroke (width 0) (type solid) (color 0 0 0 0))
@@
     (stroke (width 0) (type solid) (color 0 0 0 0))
   )
+  (wire (pts (xy 31.75 156.21) (xy 33.02 156.21))
+    (stroke (width 0) (type solid) (color 0 0 0 0))
+  )
   (wire (pts (xy 34.29 30.48) (xy 34.29 34.29))
     (stroke (width 0) (type solid) (color 0 0 0 0))
@@
     (stroke (width 0) (type solid) (color 0 0 0 0))
   )
+  (wire (pts (xy 39.37 160.02) (xy 39.37 161.29))
+    (stroke (width 0) (type solid) (color 0 0 0 0))
+  )
+  (wire (pts (xy 39.37 161.29) (xy 40.64 161.29))
+    (stroke (width 0) (type solid) (color 0 0 0 0))
+  )
   (wire (pts (xy 44.45 34.29) (xy 46.99 34.29))
     (stroke (width 0) (type solid) (color 0 0 0 0))
@@
     (stroke (width 0) (type solid) (color 0 0 0 0))
   )
-  (wire (pts (xy 44.45 153.67) (xy 46.99 153.67))
-    (stroke (width 0) (type solid) (color 0 0 0 0))
-  )
   (wire (pts (xy 45.72 30.48) (xy 46.99 30.48))
     (stroke (width 0) (type solid) (color 0 0 0 0))
@@
     (stroke (width 0) (type solid) (color 0 0 0 0))
   )
-  (wire (pts (xy 45.72 157.48) (xy 46.99 157.48))
+  (wire (pts (xy 45.72 156.21) (xy 46.99 156.21))
     (stroke (width 0) (type solid) (color 0 0 0 0))
   )
@@
   )
   (wire (pts (xy 46.99 34.29) (xy 46.99 36.83))
-    (stroke (width 0) (type solid) (color 0 0 0 0))
-  )
-  (wire (pts (xy 46.99 153.67) (xy 46.99 157.48))
-    (stroke (width 0) (type solid) (color 0 0 0 0))
-  )
-  (wire (pts (xy 46.99 153.67) (xy 48.26 153.67))
-    (stroke (width 0) (type solid) (color 0 0 0 0))
-  )
-  (polyline (pts (xy 20.32 162.56) (xy 20.32 146.05))
-    (stroke (width 0) (type solid) (color 0 0 0 0))
-  )
-  (polyline (pts (xy 20.32 162.56) (xy 21.59 162.56))
-    (stroke (width 0) (type solid) (color 0 0 0 0))
-  )
-  (polyline (pts (xy 21.59 146.05) (xy 20.32 146.05))
-    (stroke (width 0) (type solid) (color 0 0 0 0))
-  )
-  (polyline (pts (xy 21.59 146.05) (xy 60.96 146.05))
-    (stroke (width 0) (type solid) (color 0 0 0 0))
-  )
-  (polyline (pts (xy 60.96 146.05) (xy 60.96 162.56))
-    (stroke (width 0) (type solid) (color 0 0 0 0))
-  )
-  (polyline (pts (xy 60.96 162.56) (xy 21.59 162.56))
     (stroke (width 0) (type solid) (color 0 0 0 0))
   )
@@
     (effects (font (size 1.27 1.27)) (justify left bottom))
   )
-  (label "+3.3v" (at 30.48 153.67 180)
-    (effects (font (size 1.27 1.27)) (justify right bottom))
-  )
-  (label "+1.8v" (at 30.48 157.48 180)
+  (label "+3.3v" (at 31.75 156.21 180)
     (effects (font (size 1.27 1.27)) (justify right bottom))
   )
@@
   (label "WL_nDis" (at 35.56 97.79 180)
     (effects (font (size 1.27 1.27)) (justify right bottom))
+  )
+  (label "+1.8v" (at 46.99 156.21 0)
+    (effects (font (size 1.27 1.27)) (justify left bottom))
   )
   (hierarchical_label "nRPIBOOT" (shape output) (at 22.86 30.48 180)
@@
     (effects (font (size 1.27 1.27)) (justify left))
   )
-  (hierarchical_label "GPIO_VREF" (shape output) (at 48.26 153.67 0)
+  (hierarchical_label "GPIO_VREF" (shape output) (at 40.64 161.29 0)
     (effects (font (size 1.27 1.27)) (justify left))
   )
@@
   (symbol (lib_id "power:GND") (at 39.37 133.35 0) (unit 1)
     (in_bom yes) (on_board yes) (fields_autoplaced)
-    (property "Reference" "#PWR058" (id 0) (at 39.37 139.7 0)
+    (property "Reference" "#PWR062" (id 0) (at 39.37 139.7 0)
       (effects (font (size 1.27 1.27)) hide)
     )
@@
   (symbol (lib_id "power:GND") (at 46.99 36.83 0) (unit 1)
     (in_bom yes) (on_board yes)
-    (property "Reference" "#PWR062" (id 0) (at 46.99 43.18 0)
+    (property "Reference" "#PWR058" (id 0) (at 46.99 43.18 0)
       (effects (font (size 1.27 1.27)) hide)
     )
@@
     (pin "1")
   )
-  (symbol (lib_id "Jumper:Jumper_2_Bridged") (at 39.37 153.67 0) (unit 1)
-    (in_bom yes) (on_board yes)
-    (property "Reference" "JP1" (id 0) (at 39.37 148.59 0))
-    (property "Value" "Jumper_2_Bridged" (id 1) (at 39.37 151.13 0))
-    (property "Footprint" "Jumper:SolderJumper-2_P1.3mm_Bridged_Pad1.0x1.5mm" (id 2) (at 39.37 153.67 0)
-      (effects (font (size 1.27 1.27)) hide)
-    )
-    (property "Datasheet" "~" (id 3) (at 39.37 153.67 0)
-      (effects (font (size 1.27 1.27)) hide)
-    )
-    (pin "1")
-    (pin "2")
-  )
   (symbol (lib_id "Jumper:SolderJumper_2_Open") (at 40.64 34.29 0) (unit 1)
     (in_bom yes) (on_board yes) (fields_autoplaced)
-    (property "Reference" "JP2" (id 0) (at 40.64 29.21 0))
-    (property "Value" "SolderJumper_2_Open" (id 1) (at 40.64 31.75 0))
-    (property "Footprint" "Jumper:SolderJumper-2_P1.3mm_Open_TrianglePad1.0x1.5mm" (id 2) (at 40.64 34.29 0)
+    (property "Reference" "JP1" (id 0) (at 40.64 29.21 0))
+    (property "Value" "SolderJumper_2_Open" (id 1) (at 40.64 31.75 0)
+      (effects (font (size 1.27 1.27)) hide)
+    )
+    (property "Footprint" "Jumper:SolderJumper-2_P1.3mm_Open_RoundedPad1.0x1.5mm" (id 2) (at 40.64 34.29 0)
       (effects (font (size 1.27 1.27)) hide)
     )
@@
   (symbol (lib_id "Jumper:SolderJumper_2_Open") (at 40.64 66.04 0) (unit 1)
     (in_bom yes) (on_board yes) (fields_autoplaced)
-    (property "Reference" "JP3" (id 0) (at 40.64 60.96 0))
+    (property "Reference" "JP2" (id 0) (at 40.64 60.96 0))
     (property "Value" "SolderJumper_2_Open" (id 1) (at 40.64 63.5 0))
-    (property "Footprint" "Jumper:SolderJumper-2_P1.3mm_Open_TrianglePad1.0x1.5mm" (id 2) (at 40.64 66.04 0)
+    (property "Footprint" "Jumper:SolderJumper-2_P1.3mm_Open_RoundedPad1.0x1.5mm" (id 2) (at 40.64 66.04 0)
       (effects (font (size 1.27 1.27)) hide)
     )
@@
   (symbol (lib_id "Jumper:SolderJumper_2_Open") (at 40.64 83.82 0) (unit 1)
     (in_bom yes) (on_board yes) (fields_autoplaced)
-    (property "Reference" "JP4" (id 0) (at 40.64 78.74 0))
+    (property "Reference" "JP3" (id 0) (at 40.64 78.74 0))
     (property "Value" "SolderJumper_2_Open" (id 1) (at 40.64 81.28 0))
-    (property "Footprint" "Jumper:SolderJumper-2_P1.3mm_Open_TrianglePad1.0x1.5mm" (id 2) (at 40.64 83.82 0)
+    (property "Footprint" "Jumper:SolderJumper-2_P1.3mm_Open_RoundedPad1.0x1.5mm" (id 2) (at 40.64 83.82 0)
       (effects (font (size 1.27 1.27)) hide)
     )
@@
   (symbol (lib_id "Jumper:SolderJumper_2_Open") (at 40.64 97.79 0) (unit 1)
     (in_bom yes) (on_board yes)
-    (property "Reference" "JP5" (id 0) (at 40.64 92.71 0))
+    (property "Reference" "JP4" (id 0) (at 40.64 92.71 0))
     (property "Value" "SolderJumper_2_Open" (id 1) (at 40.64 95.25 0))
-    (property "Footprint" "Jumper:SolderJumper-2_P1.3mm_Open_TrianglePad1.0x1.5mm" (id 2) (at 40.64 97.79 0)
+    (property "Footprint" "Jumper:SolderJumper-2_P1.3mm_Open_RoundedPad1.0x1.5mm" (id 2) (at 40.64 97.79 0)
       (effects (font (size 1.27 1.27)) hide)
     )
     (property "Datasheet" "~" (id 3) (at 40.64 97.79 0)
-      (effects (font (size 1.27 1.27)) hide)
-    )
-    (pin "1")
-    (pin "2")
-  )
-  (symbol (lib_id "Jumper:SolderJumper_2_Open") (at 41.91 157.48 0) (unit 1)
-    (in_bom yes) (on_board yes)
-    (property "Reference" "JP6" (id 0) (at 41.91 152.4 0))
-    (property "Value" "SolderJumper_2_Open" (id 1) (at 41.91 154.94 0))
-    (property "Footprint" "Jumper:SolderJumper-2_P1.3mm_Open_TrianglePad1.0x1.5mm" (id 2) (at 41.91 157.48 0)
-      (effects (font (size 1.27 1.27)) hide)
-    )
-    (property "Datasheet" "~" (id 3) (at 41.91 157.48 0)
       (effects (font (size 1.27 1.27)) hide)
     )
@@
   (symbol (lib_id "Switch:SW_SPST") (at 33.02 123.19 0) (unit 1)
     (in_bom yes) (on_board yes) (fields_autoplaced)
-    (property "Reference" "SW1" (id 0) (at 33.02 118.11 0))
+    (property "Reference" "SW2" (id 0) (at 33.02 118.11 0))
     (property "Value" "SW_SPST" (id 1) (at 33.02 120.65 0))
     (property "Footprint" "cm4crypto:cus-12b" (id 2) (at 33.02 123.19 0)
@@
   (symbol (lib_id "Switch:SW_Push") (at 40.64 30.48 0) (unit 1)
     (in_bom yes) (on_board yes) (fields_autoplaced)
-    (property "Reference" "SW2" (id 0) (at 40.64 24.13 0))
+    (property "Reference" "SW1" (id 0) (at 40.64 24.13 0))
     (property "Value" "SW_Push" (id 1) (at 40.64 26.67 0))
     (property "Footprint" "cm4crypto:EVQ-P7C01P" (id 2) (at 40.64 25.4 0)
@@
     (pin "2")
   )
+  (symbol (lib_id "Jumper:Jumper_3_Bridged12") (at 39.37 156.21 0) (unit 1)
+    (in_bom yes) (on_board yes) (fields_autoplaced)
+    (property "Reference" "JP5" (id 0) (at 39.37 151.13 0))
+    (property "Value" "Jumper_3_Bridged12" (id 1) (at 39.37 153.67 0))
+    (property "Footprint" "Jumper:SolderJumper-3_P1.3mm_Bridged12_RoundedPad1.0x1.5mm" (id 2) (at 39.37 156.21 0)
+      (effects (font (size 1.27 1.27)) hide)
+    )
+    (property "Datasheet" "~" (id 3) (at 39.37 156.21 0)
+      (effects (font (size 1.27 1.27)) hide)
+    )
+    (pin "1")
+    (pin "2")
+    (pin "3")
+  )
 )
