File: hardware/lobby/sheets/jumpers.kicad_sch (KiCad schematic)
At the start: 8 parts, among them SW1 SW_Push, SW2 SW_SPST

Commit message: update lobby
Parts:
- renumbered R6 to R8
Changed lines of the file:
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@@
   (symbol (lib_id "power:GND") (at 39.37 133.35 0) (unit 1)
     (in_bom yes) (on_board yes) (fields_autoplaced)
-    (property "Reference" "#PWR062" (id 0) (at 39.37 139.7 0)
+    (property "Reference" "#PWR061" (id 0) (at 39.37 139.7 0)
       (effects (font (size 1.27 1.27)) hide)
     )
@@
   (symbol (lib_id "power:GND") (at 45.72 67.31 0) (unit 1)
     (in_bom yes) (on_board yes)
-    (property "Reference" "#PWR059" (id 0) (at 45.72 73.66 0)
+    (property "Reference" "#PWR058" (id 0) (at 45.72 73.66 0)
       (effects (font (size 1.27 1.27)) hide)
     )
@@
   (symbol (lib_id "power:GND") (at 45.72 85.09 0) (unit 1)
     (in_bom yes) (on_board yes)
-    (property "Reference" "#PWR060" (id 0) (at 45.72 91.44 0)
+    (property "Reference" "#PWR059" (id 0) (at 45.72 91.44 0)
       (effects (font (size 1.27 1.27)) hide)
     )
@@
   (symbol (lib_id "power:GND") (at 45.72 99.06 0) (unit 1)
     (in_bom yes) (on_board yes)
-    (property "Reference" "#PWR061" (id 0) (at 45.72 105.41 0)
+    (property "Reference" "#PWR060" (id 0) (at 45.72 105.41 0)
       (effects (font (size 1.27 1.27)) hide)
     )
@@
   (symbol (lib_id "power:GND") (at 46.99 36.83 0) (unit 1)
     (in_bom yes) (on_board yes)
-    (property "Reference" "#PWR058" (id 0) (at 46.99 43.18 0)
+    (property "Reference" "#PWR057" (id 0) (at 46.99 43.18 0)
       (effects (font (size 1.27 1.27)) hide)
     )
@@
   (symbol (lib_id "Device:R") (at 39.37 128.27 0) (unit 1)
     (in_bom yes) (on_board yes) (fields_autoplaced)
-    (property "Reference" "R6" (id 0) (at 41.91 127.6349 0)
+    (property "Reference" "R8" (id 0) (at 41.91 127.6349 0)
       (effects (font (size 1.27 1.27)) (justify left))
     )
