File: hardware/lobby/sheets/sd.kicad_sch (KiCad schematic)
At the start: 6 parts

Commit message: start routing mezzanine
making a progress capture before trying to cram a lot of signals onto just one hirose connector...
Parts:
- J1: renamed from J?; footprint CM4IO:SDCARD_MOLEX_503398-1892 -> cm4crypto:SDCARD_MOLEX_503398-1892
- gave numbers to parts that had none: 5
Changed lines of the file:
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@@
   (symbol (lib_id "power:GND") (at 97.79 85.09 0) (unit 1)
     (in_bom yes) (on_board yes)
-    (property "Reference" "#PWR?" (id 0) (at 97.79 91.44 0)
+    (property "Reference" "#PWR052" (id 0) (at 97.79 91.44 0)
       (effects (font (size 1.27 1.27)) hide)
     )
@@
   (symbol (lib_id "power:GND") (at 144.78 133.35 0) (unit 1)
     (in_bom yes) (on_board yes)
-    (property "Reference" "#PWR?" (id 0) (at 144.78 139.7 0)
+    (property "Reference" "#PWR054" (id 0) (at 144.78 139.7 0)
       (effects (font (size 1.27 1.27)) hide)
     )
@@
   (symbol (lib_id "power:GND") (at 182.88 99.06 0) (unit 1)
     (in_bom yes) (on_board yes)
-    (property "Reference" "#PWR?" (id 0) (at 182.88 105.41 0)
+    (property "Reference" "#PWR053" (id 0) (at 182.88 105.41 0)
       (effects (font (size 1.27 1.27)) hide)
     )
@@
   (symbol (lib_id "Device:R") (at 133.35 91.44 90) (unit 1)
     (in_bom yes) (on_board yes)
-    (property "Reference" "R?" (id 0) (at 132.08 93.98 90)
+    (property "Reference" "R3" (id 0) (at 132.08 93.98 90)
       (effects (font (size 1.27 1.27)) (justify left))
     )
@@
   (symbol (lib_id "Device:R") (at 133.35 99.06 90) (unit 1)
     (in_bom yes) (on_board yes)
-    (property "Reference" "R?" (id 0) (at 131.8006 101.4476 90)
+    (property "Reference" "R4" (id 0) (at 131.8006 101.4476 90)
       (effects (font (size 1.27 1.27)) (justify left))
     )
@@
   (symbol (lib_id "Device:R") (at 180.34 119.38 0) (unit 1)
     (in_bom yes) (on_board yes)
-    (property "Reference" "R?" (id 0) (at 182.118 118.2116 0)
+    (property "Reference" "R5" (id 0) (at 182.118 118.2116 0)
       (effects (font (size 1.27 1.27)) (justify left))
     )
@@
   (symbol (lib_id "Device:C") (at 97.79 77.47 0) (unit 1)
     (in_bom yes) (on_board yes)
-    (property "Reference" "C?" (id 0) (at 100.711 76.3016 0)
+    (property "Reference" "C1" (id 0) (at 100.711 76.3016 0)
       (effects (font (size 1.27 1.27)) (justify left))
     )
@@
   (symbol (lib_id "CM4IO:RT9742GGJ5") (at 156.21 132.08 0) (unit 1)
     (in_bom yes) (on_board yes)
-    (property "Reference" "U?" (id 0) (at 154.94 115.189 0))
+    (property "Reference" "U1" (id 0) (at 154.94 115.189 0))
     (property "Value" "RT9742GGJ5" (id 1) (at 154.94 117.5004 0))
     (property "Footprint" "Package_TO_SOT_SMD:SOT-23-5" (id 2) (at 156.21 132.08 0)
@@
   (symbol (lib_id "Connector:Micro_SD_Card_Det") (at 160.02 81.28 0) (unit 1)
     (in_bom yes) (on_board yes)
-    (property "Reference" "J?" (id 0) (at 158.75 60.5282 0))
+    (property "Reference" "J1" (id 0) (at 158.75 60.5282 0))
     (property "Value" "Micro_SD_Card_Det" (id 1) (at 158.75 62.8396 0))
-    (property "Footprint" "CM4IO:SDCARD_MOLEX_503398-1892" (id 2) (at 212.09 63.5 0)
-      (effects (font (size 1.27 1.27)) hide)
-    )
+    (property "Footprint" "cm4crypto:SDCARD_MOLEX_503398-1892" (id 2) (at 212.09 63.5 0)
+      (effects (font (size 1.27 1.27)) hide)
+    )

Commit message: work abroad
did some light planning for the lobby board while on vacation. now ready for final placement + routing
Parts:
- added C1: 2.2uF, Capacitor_SMD:C_0603_1608Metric, symbol Device:C
- added C2: 0.1uF, Capacitor_SMD:C_0603_1608Metric, symbol Device:C
- C3: renamed from C1; footprint Capacitor_SMD:C_0805_2012Metric -> Capacitor_SMD:C_0603_1608Metric
- R3, R4: footprint Resistor_SMD:R_0402_1005Metric -> Resistor_SMD:R_0603_1608Metric
- renumbered J1 to J3
Connections:
- net +3.3v: now also C1.1, C2.1
- net GND: now also C1.2, C2.2
Changed lines of the file:
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@@
 (kicad_sch (version 20210406) (generator eeschema)
   (paper "A4")
+  (junction (at 86.36 107.95) (diameter 1.016) (color 0 0 0 0))
+  (junction (at 86.36 115.57) (diameter 1.016) (color 0 0 0 0))
   (junction (at 97.79 72.39) (diameter 0.9144) (color 0 0 0 0))
   (junction (at 97.79 83.82) (diameter 0.9144) (color 0 0 0 0))
@@
   (junction (at 180.34 127) (diameter 0.9144) (color 0 0 0 0))
   (no_connect (at 147.32 127))
+  (wire (pts (xy 80.01 107.95) (xy 86.36 107.95))
+    (stroke (width 0) (type solid) (color 0 0 0 0))
+  )
+  (wire (pts (xy 86.36 107.95) (xy 95.504 107.95))
+    (stroke (width 0) (type solid) (color 0 0 0 0))
+  )
+  (wire (pts (xy 86.36 115.57) (xy 95.504 115.57))
+    (stroke (width 0) (type solid) (color 0 0 0 0))
+  )
+  (wire (pts (xy 86.36 119.38) (xy 86.36 115.57))
+    (stroke (width 0) (type solid) (color 0 0 0 0))
+  )
   (wire (pts (xy 97.79 66.04) (xy 97.79 72.39))
     (stroke (width 0) (type solid) (color 0 0 0 0))
@@
     (effects (font (size 2.007 2.007)) (justify left bottom))
   )
+  (label "+3.3v" (at 80.01 107.95 0)
+    (effects (font (size 1.27 1.27)) (justify left bottom))
+  )
   (label "SD_PWR" (at 97.79 71.12 90)
     (effects (font (size 1.27 1.27)) (justify left bottom))
@@
     (effects (font (size 1.27 1.27)) (justify left bottom))
   )
+  (hierarchical_label "+3.3v" (shape input) (at 80.01 107.95 180)
+    (effects (font (size 1.27 1.27)) (justify right))
+  )
   (hierarchical_label "SD_DAT2" (shape bidirectional) (at 125.73 71.12 180)
     (effects (font (size 1.27 1.27)) (justify right))
@@
     (effects (font (size 1.27 1.27)) (justify left))
   )
+  (symbol (lib_id "power:GND") (at 86.36 119.38 0) (unit 1)
+    (in_bom yes) (on_board yes)
+    (property "Reference" "#PWR054" (id 0) (at 86.36 125.73 0)
+      (effects (font (size 1.27 1.27)) hide)
+    )
+    (property "Value" "GND" (id 1) (at 86.487 123.7742 0))
+    (property "Footprint" "" (id 2) (at 86.36 119.38 0)
+      (effects (font (size 1.27 1.27)) hide)
+    )
+    (property "Datasheet" "" (id 3) (at 86.36 119.38 0)
+      (effects (font (size 1.27 1.27)) hide)
+    )
+    (pin "1")
+  )
   (symbol (lib_id "power:GND") (at 97.79 85.09 0) (unit 1)
     (in_bom yes) (on_board yes)
-    (property "Reference" "#PWR?" (id 0) (at 97.79 91.44 0)
+    (property "Reference" "#PWR055" (id 0) (at 97.79 91.44 0)
       (effects (font (size 1.27 1.27)) hide)
     )
@@
   (symbol (lib_id "power:GND") (at 144.78 133.35 0) (unit 1)
     (in_bom yes) (on_board yes)
-    (property "Reference" "#PWR?" (id 0) (at 144.78 139.7 0)
+    (property "Reference" "#PWR056" (id 0) (at 144.78 139.7 0)
       (effects (font (size 1.27 1.27)) hide)
     )
@@
   (symbol (lib_id "power:GND") (at 182.88 99.06 0) (unit 1)
     (in_bom yes) (on_board yes)
-    (property "Reference" "#PWR?" (id 0) (at 182.88 105.41 0)
+    (property "Reference" "#PWR057" (id 0) (at 182.88 105.41 0)
       (effects (font (size 1.27 1.27)) hide)
     )
@@
       (effects (font (size 1.27 1.27)) (justify left))
     )
-    (property "Footprint" "Resistor_SMD:R_0402_1005Metric" (id 2) (at 133.35 93.218 90)
+    (property "Footprint" "Resistor_SMD:R_0603_1608Metric" (id 2) (at 133.35 93.218 90)
       (effects (font (size 1.27 1.27)) hide)
     )
@@
       (effects (font (size 1.27 1.27)) (justify left))
     )
-    (property "Footprint" "Resistor_SMD:R_0402_1005Metric" (id 2) (at 133.35 100.838 90)
+    (property "Footprint" "Resistor_SMD:R_0603_1608Metric" (id 2) (at 133.35 100.838 90)
       (effects (font (size 1.27 1.27)) hide)
     )
@@
     (pin "2")
   )
+  (symbol (lib_id "Device:C") (at 86.36 111.76 0) (unit 1)
+    (in_bom yes) (on_board yes)
+    (property "Reference" "C1" (id 0) (at 89.281 110.5916 0)
+      (effects (font (size 1.27 1.27)) (justify left))
+    )
+    (property "Value" "2.2uF" (id 1) (at 89.281 112.903 0)
+      (effects (font (size 1.27 1.27)) (justify left))
+    )
+    (property "Footprint" "Capacitor_SMD:C_0603_1608Metric" (id 2) (at 87.3252 115.57 0)
+      (effects (font (size 1.27 1.27)) hide)
+    )
+    (property "Datasheet" "https://search.murata.co.jp/Ceramy/image/img/A01X/G101/ENG/GRM21BR71A106KA73-01.pdf" (id 3) (at 86.36 111.76 0)
+      (effects (font (size 1.27 1.27)) hide)
+    )
+    (property "Field5" "490-14381-1-ND" (id 4) (at 86.36 111.76 0)
+      (effects (font (size 1.27 1.27)) hide)
+    )
+    (property "Field4" "Digikey" (id 5) (at 86.36 111.76 0)
+      (effects (font (size 1.27 1.27)) hide)
+    )
+    (property "Field6" "GRM21BR71A106KA73L" (id 6) (at 86.36 111.76 0)
+      (effects (font (size 1.27 1.27)) hide)
+    )
+    (property "Field7" "Murata" (id 7) (at 86.36 111.76 0)
+      (effects (font (size 1.27 1.27)) hide)
+    )
+    (property "Part Description" "	10uF 10% 10V Ceramic Capacitor X7R 0805 (2012 Metric)" (id 8) (at 86.36 111.76 0)
+      (effects (font (size 1.27 1.27)) hide)
+    )
+    (property "Field8" "111893011" (id 9) (at 86.36 111.76 0)
+      (effects (font (size 1.27 1.27)) hide)
+    )
+    (pin "1")
+    (pin "2")
+  )
+  (symbol (lib_id "Device:C") (at 95.504 111.76 0) (unit 1)
+    (in_bom yes) (on_board yes)
+    (property "Reference" "C2" (id 0) (at 98.425 110.5916 0)
+      (effects (font (size 1.27 1.27)) (justify left))
+    )
+    (property "Value" "0.1uF" (id 1) (at 98.425 112.903 0)
+      (effects (font (size 1.27 1.27)) (justify left))
+    )
+    (property "Footprint" "Capacitor_SMD:C_0603_1608Metric" (id 2) (at 96.4692 115.57 0)
+      (effects (font (size 1.27 1.27)) hide)
+    )
+    (property "Datasheet" "https://search.murata.co.jp/Ceramy/image/img/A01X/G101/ENG/GRM21BR71A106KA73-01.pdf" (id 3) (at 95.504 111.76 0)
+      (effects (font (size 1.27 1.27)) hide)
+    )
+    (property "Field5" "490-14381-1-ND" (id 4) (at 95.504 111.76 0)
+      (effects (font (size 1.27 1.27)) hide)
+    )
+    (property "Field4" "Digikey" (id 5) (at 95.504 111.76 0)
+      (effects (font (size 1.27 1.27)) hide)
+    )
+    (property "Field6" "GRM21BR71A106KA73L" (id 6) (at 95.504 111.76 0)
+      (effects (font (size 1.27 1.27)) hide)
+    )
+    (property "Field7" "Murata" (id 7) (at 95.504 111.76 0)
+      (effects (font (size 1.27 1.27)) hide)
+    )
+    (property "Part Description" "	10uF 10% 10V Ceramic Capacitor X7R 0805 (2012 Metric)" (id 8) (at 95.504 111.76 0)
+      (effects (font (size 1.27 1.27)) hide)
+    )
+    (property "Field8" "111893011" (id 9) (at 95.504 111.76 0)
+      (effects (font (size 1.27 1.27)) hide)
+    )
+    (pin "1")
+    (pin "2")
+  )
   (symbol (lib_id "Device:C") (at 97.79 77.47 0) (unit 1)
     (in_bom yes) (on_board yes)
-    (property "Reference" "C1" (id 0) (at 100.711 76.3016 0)
+    (property "Reference" "C3" (id 0) (at 100.711 76.3016 0)
       (effects (font (size 1.27 1.27)) (justify left))
     )
@@
       (effects (font (size 1.27 1.27)) (justify left))
     )
-    (property "Footprint" "Capacitor_SMD:C_0805_2012Metric" (id 2) (at 98.7552 81.28 0)
+    (property "Footprint" "Capacitor_SMD:C_0603_1608Metric" (id 2) (at 98.7552 81.28 0)
       (effects (font (size 1.27 1.27)) hide)
     )
@@
   (symbol (lib_id "Connector:Micro_SD_Card_Det") (at 160.02 81.28 0) (unit 1)
     (in_bom yes) (on_board yes)
-    (property "Reference" "J1" (id 0) (at 158.75 60.5282 0))
+    (property "Reference" "J3" (id 0) (at 158.75 60.5282 0))
     (property "Value" "Micro_SD_Card_Det" (id 1) (at 158.75 62.8396 0))
     (property "Footprint" "cm4crypto:SDCARD_MOLEX_503398-1892" (id 2) (at 212.09 63.5 0)

Commit message: place lobby components
Parts:
- R5: footprint Resistor_SMD:R_0402_1005Metric -> Resistor_SMD:R_0603_1608Metric
- renumbered C3 to C1, C1 to C2, C2 to C3
Changed lines of the file:
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@@
   (symbol (lib_id "power:GND") (at 86.36 119.38 0) (unit 1)
     (in_bom yes) (on_board yes)
-    (property "Reference" "#PWR054" (id 0) (at 86.36 125.73 0)
+    (property "Reference" "#PWR056" (id 0) (at 86.36 125.73 0)
       (effects (font (size 1.27 1.27)) hide)
     )
@@
   (symbol (lib_id "power:GND") (at 97.79 85.09 0) (unit 1)
     (in_bom yes) (on_board yes)
-    (property "Reference" "#PWR055" (id 0) (at 97.79 91.44 0)
+    (property "Reference" "#PWR054" (id 0) (at 97.79 91.44 0)
       (effects (font (size 1.27 1.27)) hide)
     )
@@
   (symbol (lib_id "power:GND") (at 144.78 133.35 0) (unit 1)
     (in_bom yes) (on_board yes)
-    (property "Reference" "#PWR056" (id 0) (at 144.78 139.7 0)
+    (property "Reference" "#PWR057" (id 0) (at 144.78 139.7 0)
       (effects (font (size 1.27 1.27)) hide)
     )
@@
   (symbol (lib_id "power:GND") (at 182.88 99.06 0) (unit 1)
     (in_bom yes) (on_board yes)
-    (property "Reference" "#PWR057" (id 0) (at 182.88 105.41 0)
+    (property "Reference" "#PWR055" (id 0) (at 182.88 105.41 0)
       (effects (font (size 1.27 1.27)) hide)
     )
@@
       (effects (font (size 1.27 1.27)) (justify left))
     )
-    (property "Footprint" "Resistor_SMD:R_0402_1005Metric" (id 2) (at 178.562 119.38 90)
+    (property "Footprint" "Resistor_SMD:R_0603_1608Metric" (id 2) (at 178.562 119.38 90)
       (effects (font (size 1.27 1.27)) hide)
     )
@@
   (symbol (lib_id "Device:C") (at 86.36 111.76 0) (unit 1)
     (in_bom yes) (on_board yes)
-    (property "Reference" "C1" (id 0) (at 89.281 110.5916 0)
+    (property "Reference" "C2" (id 0) (at 89.281 110.5916 0)
       (effects (font (size 1.27 1.27)) (justify left))
     )
@@
   (symbol (lib_id "Device:C") (at 95.504 111.76 0) (unit 1)
     (in_bom yes) (on_board yes)
-    (property "Reference" "C2" (id 0) (at 98.425 110.5916 0)
+    (property "Reference" "C3" (id 0) (at 98.425 110.5916 0)
       (effects (font (size 1.27 1.27)) (justify left))
     )
@@
   (symbol (lib_id "Device:C") (at 97.79 77.47 0) (unit 1)
     (in_bom yes) (on_board yes)
-    (property "Reference" "C3" (id 0) (at 100.711 76.3016 0)
-      (effects (font (size 1.27 1.27)) (justify left))
-    )
+    (property "Reference" "C1" (id 0) (at 100.711 76.3016 0)
+      (effects (font (size 1.27 1.27)) (justify left))
+    )

Commit message: update lobby
Parts:
- J3: footprint cm4crypto:SDCARD_MOLEX_503398-1892 -> cm4crypto:amphenol-sd-push-pull_114-00841-68
- renumbered R3 to R5, R4 to R6, R5 to R7
Changed lines of the file:
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@@
   (symbol (lib_id "power:GND") (at 86.36 119.38 0) (unit 1)
     (in_bom yes) (on_board yes)
-    (property "Reference" "#PWR056" (id 0) (at 86.36 125.73 0)
+    (property "Reference" "#PWR055" (id 0) (at 86.36 125.73 0)
       (effects (font (size 1.27 1.27)) hide)
     )
@@
   (symbol (lib_id "power:GND") (at 97.79 85.09 0) (unit 1)
     (in_bom yes) (on_board yes)
-    (property "Reference" "#PWR054" (id 0) (at 97.79 91.44 0)
+    (property "Reference" "#PWR053" (id 0) (at 97.79 91.44 0)
       (effects (font (size 1.27 1.27)) hide)
     )
@@
   (symbol (lib_id "power:GND") (at 144.78 133.35 0) (unit 1)
     (in_bom yes) (on_board yes)
-    (property "Reference" "#PWR057" (id 0) (at 144.78 139.7 0)
+    (property "Reference" "#PWR056" (id 0) (at 144.78 139.7 0)
       (effects (font (size 1.27 1.27)) hide)
     )
@@
   (symbol (lib_id "power:GND") (at 182.88 99.06 0) (unit 1)
     (in_bom yes) (on_board yes)
-    (property "Reference" "#PWR055" (id 0) (at 182.88 105.41 0)
+    (property "Reference" "#PWR054" (id 0) (at 182.88 105.41 0)
       (effects (font (size 1.27 1.27)) hide)
     )
@@
   (symbol (lib_id "Device:R") (at 133.35 91.44 90) (unit 1)
     (in_bom yes) (on_board yes)
-    (property "Reference" "R3" (id 0) (at 132.08 93.98 90)
+    (property "Reference" "R5" (id 0) (at 132.08 93.98 90)
       (effects (font (size 1.27 1.27)) (justify left))
     )
@@
       (effects (font (size 1.27 1.27)) hide)
     )
-    (property "Datasheet" "https://fscdn.rohm.com/en/products/databook/datasheet/passive/resistor/chip_resistor/mcr-e.pdf" (id 3) (at 133.35 91.44 0)
+    (property "Datasheet" "~" (id 3) (at 133.35 91.44 0)
       (effects (font (size 1.27 1.27)) hide)
     )
@@
   (symbol (lib_id "Device:R") (at 133.35 99.06 90) (unit 1)
     (in_bom yes) (on_board yes)
-    (property "Reference" "R4" (id 0) (at 131.8006 101.4476 90)
+    (property "Reference" "R6" (id 0) (at 131.8006 101.4476 90)
       (effects (font (size 1.27 1.27)) (justify left))
     )
@@
       (effects (font (size 1.27 1.27)) hide)
     )
-    (property "Datasheet" "https://fscdn.rohm.com/en/products/databook/datasheet/passive/resistor/chip_resistor/mcr-e.pdf" (id 3) (at 133.35 99.06 0)
+    (property "Datasheet" "~" (id 3) (at 133.35 99.06 0)
       (effects (font (size 1.27 1.27)) hide)
     )
@@
   (symbol (lib_id "Device:R") (at 180.34 119.38 0) (unit 1)
     (in_bom yes) (on_board yes)
-    (property "Reference" "R5" (id 0) (at 182.118 118.2116 0)
+    (property "Reference" "R7" (id 0) (at 182.118 118.2116 0)
       (effects (font (size 1.27 1.27)) (justify left))
     )
@@
       (effects (font (size 1.27 1.27)) hide)
     )
-    (property "Datasheet" "https://fscdn.rohm.com/en/products/databook/datasheet/passive/resistor/chip_resistor/mcr-e.pdf" (id 3) (at 180.34 119.38 0)
+    (property "Datasheet" "~" (id 3) (at 180.34 119.38 0)
       (effects (font (size 1.27 1.27)) hide)
     )
@@
       (effects (font (size 1.27 1.27)) hide)
     )
-    (property "Datasheet" "https://search.murata.co.jp/Ceramy/image/img/A01X/G101/ENG/GRM21BR71A106KA73-01.pdf" (id 3) (at 86.36 111.76 0)
+    (property "Datasheet" "~" (id 3) (at 86.36 111.76 0)
       (effects (font (size 1.27 1.27)) hide)
     )
@@
       (effects (font (size 1.27 1.27)) hide)
     )
-    (property "Datasheet" "https://search.murata.co.jp/Ceramy/image/img/A01X/G101/ENG/GRM21BR71A106KA73-01.pdf" (id 3) (at 95.504 111.76 0)
+    (property "Datasheet" "~" (id 3) (at 95.504 111.76 0)
       (effects (font (size 1.27 1.27)) hide)
     )
@@
       (effects (font (size 1.27 1.27)) hide)
     )
-    (property "Datasheet" "https://search.murata.co.jp/Ceramy/image/img/A01X/G101/ENG/GRM21BR71A106KA73-01.pdf" (id 3) (at 97.79 77.47 0)
+    (property "Datasheet" "~" (id 3) (at 97.79 77.47 0)
       (effects (font (size 1.27 1.27)) hide)
     )
@@
     (property "Reference" "J3" (id 0) (at 158.75 60.5282 0))
     (property "Value" "Micro_SD_Card_Det" (id 1) (at 158.75 62.8396 0))
-    (property "Footprint" "cm4crypto:SDCARD_MOLEX_503398-1892" (id 2) (at 212.09 63.5 0)
-      (effects (font (size 1.27 1.27)) hide)
-    )
+    (property "Footprint" "cm4crypto:amphenol-sd-push-pull_114-00841-68" (id 2) (at 212.09 63.5 0)
+      (effects (font (size 1.27 1.27)) hide)
+    )
