File: hardware/lobby/sheets/_autosave-jumpers.kicad_sch (KiCad schematic)
At the start: 8 parts, among them SW2 SW_SPST

Commit message: update silkscreen
Parts:
- gave numbers to parts that had none: 1
Changed lines of the file:
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@@
   (symbol (lib_id "Switch:SW_SPST") (at 40.64 30.48 0) (unit 1)
     (in_bom yes) (on_board yes) (fields_autoplaced)
-    (property "Reference" "SW?" (id 0) (at 40.64 25.4 0))
+    (property "Reference" "SW1" (id 0) (at 40.64 25.4 0))
     (property "Value" "SW_SPST" (id 1) (at 40.64 27.94 0))
     (property "Footprint" "cm4crypto:cus-12b" (id 2) (at 40.64 30.48 0)
