File: hardware/lobby/sheets/usb-mux.kicad_sch (KiCad schematic)
At the start: 1 part

Commit message: start routing mezzanine
making a progress capture before trying to cram a lot of signals onto just one hirose connector...
Parts:
- U4: renamed from U?; footprint (none) -> Package_SO:MSOP-10_3x3mm_P0.5mm
Changed lines of the file:
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@@
   (symbol (lib_id "power:GND") (at 143.51 105.41 0) (unit 1)
     (in_bom yes) (on_board yes) (fields_autoplaced)
-    (property "Reference" "#PWR?" (id 0) (at 143.51 111.76 0)
+    (property "Reference" "#PWR0116" (id 0) (at 143.51 111.76 0)
       (effects (font (size 1.27 1.27)) hide)
     )
@@
   (symbol (lib_id "cm4crypto:FSUSB42MX") (at 153.67 105.41 0) (mirror y) (unit 1)
     (in_bom yes) (on_board yes) (fields_autoplaced)
-    (property "Reference" "U?" (id 0) (at 154.94 82.55 0))
+    (property "Reference" "U4" (id 0) (at 154.94 82.55 0))
     (property "Value" "FSUSB42MX" (id 1) (at 154.94 85.09 0))
-    (property "Footprint" "" (id 2) (at 153.67 105.41 0)
+    (property "Footprint" "Package_SO:MSOP-10_3x3mm_P0.5mm" (id 2) (at 153.67 105.41 0)
       (effects (font (size 1.27 1.27)) hide)
     )

Commit message: sheet refs relative, copied escalator pinout to lobby
Parts:
- renumbered U4 to U?
Changed lines of the file:
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@@
   (symbol (lib_id "power:GND") (at 143.51 105.41 0) (unit 1)
     (in_bom yes) (on_board yes) (fields_autoplaced)
-    (property "Reference" "#PWR0116" (id 0) (at 143.51 111.76 0)
+    (property "Reference" "#PWR?" (id 0) (at 143.51 111.76 0)
       (effects (font (size 1.27 1.27)) hide)
     )
@@
   (symbol (lib_id "cm4crypto:FSUSB42MX") (at 153.67 105.41 0) (mirror y) (unit 1)
     (in_bom yes) (on_board yes) (fields_autoplaced)
-    (property "Reference" "U4" (id 0) (at 154.94 82.55 0))
+    (property "Reference" "U?" (id 0) (at 154.94 82.55 0))
     (property "Value" "FSUSB42MX" (id 1) (at 154.94 85.09 0))
     (property "Footprint" "Package_SO:MSOP-10_3x3mm_P0.5mm" (id 2) (at 153.67 105.41 0)

Commit message: work abroad
did some light planning for the lobby board while on vacation. now ready for final placement + routing
Parts:
- added C8: 2.2uF, Capacitor_SMD:C_0603_1608Metric, symbol Device:C
- added C9: 0.1uF, Capacitor_SMD:C_0603_1608Metric, symbol Device:C
- gave numbers to parts that had none: 1
Connections:
- net +3.3v: now also C8.1, C9.1
- net GND: now also C8.2, C9.2
Other:
- note added: "USB2_DEV should go to the type-c port"
- note added: "USB2_HOST should go to type-A port"
- note added: "the usb-c port can be used as an otg "device" port. this option must be selected by the user and is exclusive of "host" functions on the A port this is the intended method of flashing firmware onto the cm4"
- note removed: "USB2_DEV should go to the type-c port (route via unused pins on hirose connectors)"
- note removed: "USB2_HOST should go to type-A port (route through standard cm4 usb pins on hirose connector)"
- note removed: "the usb-c port can be used as an otg "device" port. this option must be selected by the user and is exclusive of "host" functions on the A port"
Changed lines of the file:
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@@
 (kicad_sch (version 20210406) (generator eeschema)
   (paper "A4")
+  (junction (at 101.6 90.17) (diameter 1.016) (color 0 0 0 0))
+  (junction (at 101.6 97.79) (diameter 1.016) (color 0 0 0 0))
   (junction (at 143.51 104.14) (diameter 0.9144) (color 0 0 0 0))
+  (wire (pts (xy 95.25 90.17) (xy 101.6 90.17))
+    (stroke (width 0) (type solid) (color 0 0 0 0))
+  )
+  (wire (pts (xy 101.6 90.17) (xy 110.744 90.17))
+    (stroke (width 0) (type solid) (color 0 0 0 0))
+  )
+  (wire (pts (xy 101.6 97.79) (xy 110.744 97.79))
+    (stroke (width 0) (type solid) (color 0 0 0 0))
+  )
+  (wire (pts (xy 101.6 101.6) (xy 101.6 97.79))
+    (stroke (width 0) (type solid) (color 0 0 0 0))
+  )
   (wire (pts (xy 140.97 91.44) (xy 144.78 91.44))
     (stroke (width 0) (type solid) (color 0 0 0 0))
@@
     (stroke (width 0) (type solid) (color 0 0 0 0))
   )
-  (text "the usb-c port can be used as an otg \"device\" port. this option must be\nselected by the user and is exclusive of \"host\" functions on the A port"
+  (text "the usb-c port can be used as an otg \"device\" port. this option must be\nselected by the user and is exclusive of \"host\" functions on the A port\n\nthis is the intended method of flashing firmware onto the cm4"
     (at 173.99 139.7 0)
-    (effects (font (size 1.27 1.27)) (justify right bottom))
-  )
-  (text "USB2_DEV should go to the type-c port\n(route via unused pins on hirose connectors)"
-    (at 186.69 104.14 0)
     (effects (font (size 1.27 1.27)) (justify left bottom))
   )
-  (text "USB2_HOST should go to type-A port\n(route through standard cm4 usb pins on hirose connector)"
-    (at 187.96 92.71 0)
+  (text "USB2_DEV should go to the type-c port" (at 186.69 104.14 0)
     (effects (font (size 1.27 1.27)) (justify left bottom))
+  )
+  (text "USB2_HOST should go to type-A port" (at 187.96 92.71 0)
+    (effects (font (size 1.27 1.27)) (justify left bottom))
+  )
+  (label "+3.3v" (at 95.25 90.17 0)
+    (effects (font (size 1.27 1.27)) (justify left bottom))
+  )
+  (hierarchical_label "+3.3v" (shape input) (at 95.25 90.17 180)
+    (effects (font (size 1.27 1.27)) (justify right))
   )
   (hierarchical_label "USBOTG_ID" (shape input) (at 140.97 91.44 180)
@@
     (effects (font (size 1.27 1.27)) (justify left))
   )
+  (symbol (lib_id "power:GND") (at 101.6 101.6 0) (unit 1)
+    (in_bom yes) (on_board yes)
+    (property "Reference" "#PWR099" (id 0) (at 101.6 107.95 0)
+      (effects (font (size 1.27 1.27)) hide)
+    )
+    (property "Value" "GND" (id 1) (at 101.727 105.9942 0))
+    (property "Footprint" "" (id 2) (at 101.6 101.6 0)
+      (effects (font (size 1.27 1.27)) hide)
+    )
+    (property "Datasheet" "" (id 3) (at 101.6 101.6 0)
+      (effects (font (size 1.27 1.27)) hide)
+    )
+    (pin "1")
+  )
   (symbol (lib_id "power:GND") (at 143.51 105.41 0) (unit 1)
     (in_bom yes) (on_board yes) (fields_autoplaced)
-    (property "Reference" "#PWR?" (id 0) (at 143.51 111.76 0)
+    (property "Reference" "#PWR0100" (id 0) (at 143.51 111.76 0)
       (effects (font (size 1.27 1.27)) hide)
     )
@@
     (pin "1")
   )
+  (symbol (lib_id "Device:C") (at 101.6 93.98 0) (unit 1)
+    (in_bom yes) (on_board yes)
+    (property "Reference" "C8" (id 0) (at 104.521 92.8116 0)
+      (effects (font (size 1.27 1.27)) (justify left))
+    )
+    (property "Value" "2.2uF" (id 1) (at 104.521 95.123 0)
+      (effects (font (size 1.27 1.27)) (justify left))
+    )
+    (property "Footprint" "Capacitor_SMD:C_0603_1608Metric" (id 2) (at 102.5652 97.79 0)
+      (effects (font (size 1.27 1.27)) hide)
+    )
+    (property "Datasheet" "https://search.murata.co.jp/Ceramy/image/img/A01X/G101/ENG/GRM21BR71A106KA73-01.pdf" (id 3) (at 101.6 93.98 0)
+      (effects (font (size 1.27 1.27)) hide)
+    )
+    (property "Field5" "490-14381-1-ND" (id 4) (at 101.6 93.98 0)
+      (effects (font (size 1.27 1.27)) hide)
+    )
+    (property "Field4" "Digikey" (id 5) (at 101.6 93.98 0)
+      (effects (font (size 1.27 1.27)) hide)
+    )
+    (property "Field6" "GRM21BR71A106KA73L" (id 6) (at 101.6 93.98 0)
+      (effects (font (size 1.27 1.27)) hide)
+    )
+    (property "Field7" "Murata" (id 7) (at 101.6 93.98 0)
+      (effects (font (size 1.27 1.27)) hide)
+    )
+    (property "Part Description" "	10uF 10% 10V Ceramic Capacitor X7R 0805 (2012 Metric)" (id 8) (at 101.6 93.98 0)
+      (effects (font (size 1.27 1.27)) hide)
+    )
+    (property "Field8" "111893011" (id 9) (at 101.6 93.98 0)
+      (effects (font (size 1.27 1.27)) hide)
+    )
+    (pin "1")
+    (pin "2")
+  )
+  (symbol (lib_id "Device:C") (at 110.744 93.98 0) (unit 1)
+    (in_bom yes) (on_board yes)
+    (property "Reference" "C9" (id 0) (at 113.665 92.8116 0)
+      (effects (font (size 1.27 1.27)) (justify left))
+    )
+    (property "Value" "0.1uF" (id 1) (at 113.665 95.123 0)
+      (effects (font (size 1.27 1.27)) (justify left))
+    )
+    (property "Footprint" "Capacitor_SMD:C_0603_1608Metric" (id 2) (at 111.7092 97.79 0)
+      (effects (font (size 1.27 1.27)) hide)
+    )
+    (property "Datasheet" "https://search.murata.co.jp/Ceramy/image/img/A01X/G101/ENG/GRM21BR71A106KA73-01.pdf" (id 3) (at 110.744 93.98 0)
+      (effects (font (size 1.27 1.27)) hide)
+    )
+    (property "Field5" "490-14381-1-ND" (id 4) (at 110.744 93.98 0)
+      (effects (font (size 1.27 1.27)) hide)
+    )
+    (property "Field4" "Digikey" (id 5) (at 110.744 93.98 0)
+      (effects (font (size 1.27 1.27)) hide)
+    )
+    (property "Field6" "GRM21BR71A106KA73L" (id 6) (at 110.744 93.98 0)
+      (effects (font (size 1.27 1.27)) hide)
+    )
+    (property "Field7" "Murata" (id 7) (at 110.744 93.98 0)
+      (effects (font (size 1.27 1.27)) hide)
+    )
+    (property "Part Description" "	10uF 10% 10V Ceramic Capacitor X7R 0805 (2012 Metric)" (id 8) (at 110.744 93.98 0)
+      (effects (font (size 1.27 1.27)) hide)
+    )
+    (property "Field8" "111893011" (id 9) (at 110.744 93.98 0)
+      (effects (font (size 1.27 1.27)) hide)
+    )
+    (pin "1")
+    (pin "2")
+  )
   (symbol (lib_id "cm4crypto:FSUSB42MX") (at 153.67 105.41 0) (mirror y) (unit 1)
     (in_bom yes) (on_board yes) (fields_autoplaced)
-    (property "Reference" "U?" (id 0) (at 154.94 82.55 0))
+    (property "Reference" "U4" (id 0) (at 154.94 82.55 0))
     (property "Value" "FSUSB42MX" (id 1) (at 154.94 85.09 0))
     (property "Footprint" "Package_SO:MSOP-10_3x3mm_P0.5mm" (id 2) (at 153.67 105.41 0)

Commit message: change fusb42mx to qfn package
Parts:
- U4: footprint Package_SO:MSOP-10_3x3mm_P0.5mm -> Package_DFN_QFN:UQFN-10_1.6x2.1mm_P0.5mm
Connections:
- net USB2_DEV_N: now also U4.6 (HSD0_M); no longer U4.8 (HSD1_M)
- net USB2_DEV_P: now also U4.7 (HSD0_P); no longer U4.9 (HSD1_P)
- net USB2_HOST_N: now also U4.8 (HSD1_M); no longer U4.6 (HSD0_M)
- net USB2_HOST_P: now also U4.9 (HSD1_P); no longer U4.7 (HSD0_P)
Changed lines of the file:
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@@
     (effects (font (size 1.27 1.27)) (justify left bottom))
   )
-  (text "USB2_DEV should go to the type-c port" (at 186.69 104.14 0)
+  (text "USB2_DEV should go to the type-c port" (at 186.69 91.44 0)
     (effects (font (size 1.27 1.27)) (justify left bottom))
   )
-  (text "USB2_HOST should go to type-A port" (at 187.96 92.71 0)
+  (text "USB2_HOST should go to type-A port" (at 187.96 105.41 0)
     (effects (font (size 1.27 1.27)) (justify left bottom))
   )
@@
     (effects (font (size 1.27 1.27)) (justify left))
   )
-  (hierarchical_label "USB2_HOST_P" (shape bidirectional) (at 168.91 88.9 0)
+  (hierarchical_label "USB2_DEV_P" (shape bidirectional) (at 168.91 88.9 0)
     (effects (font (size 1.27 1.27)) (justify left))
   )
-  (hierarchical_label "USB2_HOST_N" (shape bidirectional) (at 168.91 91.44 0)
+  (hierarchical_label "USB2_DEV_N" (shape bidirectional) (at 168.91 91.44 0)
     (effects (font (size 1.27 1.27)) (justify left))
   )
-  (hierarchical_label "USB2_DEV_P" (shape bidirectional) (at 168.91 101.6 0)
+  (hierarchical_label "USB2_HOST_P" (shape bidirectional) (at 168.91 101.6 0)
     (effects (font (size 1.27 1.27)) (justify left))
   )
-  (hierarchical_label "USB2_DEV_N" (shape bidirectional) (at 168.91 104.14 0)
+  (hierarchical_label "USB2_HOST_N" (shape bidirectional) (at 168.91 104.14 0)
     (effects (font (size 1.27 1.27)) (justify left))
   )
@@
     (property "Reference" "U4" (id 0) (at 154.94 82.55 0))
     (property "Value" "FSUSB42MX" (id 1) (at 154.94 85.09 0))
-    (property "Footprint" "Package_SO:MSOP-10_3x3mm_P0.5mm" (id 2) (at 153.67 105.41 0)
+    (property "Footprint" "Package_DFN_QFN:UQFN-10_1.6x2.1mm_P0.5mm" (id 2) (at 153.67 105.41 0)
       (effects (font (size 1.27 1.27)) hide)
     )
